File: eagle/PCB/PCB 1.brd (EAGLE design)
At the start: 45 x 75 mm, 37 parts

Commit message: PCB work
Parts:
- removed 5V, DVR5V, DVRB1, DVRB2, DVRB3, DVRGND, DVRVIN, DVRVOUT, G, GND1, K1, K2, K3, SCL, SDA, VDVR, VMAIN, VMOD: (no value), wirepad:SMD1,27-2,54
- removed FTDI: (no value), pinhead:1X06
- removed GND-O, VCC-IN: (no value), wirepad:2,54/1,1
- added IO1, IO2: (no value), con-lstb:MA07-1
- added IO3: (no value), con-lstb:MA04-1
- added V-IN: (no value), wirepad:2,54/1,1
- GND: device wirepad:SMD1,27-2,54 -> wirepad:2,54/1,1
- moved VCC-O 21.8 mm to (7.62, 59.7)
- moved GND 16.5 mm to (2.54, 12.7)
- moved 8V-O 14.5 mm to (22.9, 11.4)
- moved MINIMOSD 5.24 mm to (21.6, 25.4), turned to 180 degrees
- moved GND-IN 3.81 mm to (22.9, 72.4)
- moved 3.5MM 2.54 mm to (29.2, 0.00)
- moved RJ45 2.54 mm to (12.7, 2.54)
- moved DC-JACK 1.80 mm to (8.89, 66.0)
- moved ADRUINO-NANO 1.27 mm to (31.8, 49.5)
- turned BUZZ to 270 degrees
Connections:
- net RAW renamed BAT1
- net RAWGND renamed BGND
- removed net N$1: ADRUINO-NANO.GND1, BUZZ.-, GND.1, GND1.1
- removed net N$18: ADRUINO-NANO.3.3V, ADRUINO-NANO.A0, R1.1, R2.2
- new net HP1: ADRUINO-NANO.A4, IO2.1
- new net HP2: ADRUINO-NANO.A5, IO2.2
- new net HP3: -OUT.1, 3.5MM.1, ADRUINO-NANO.GND, BUZZ.-, IO1.3, IO2.3, IO3.1, MINIMOSD.IGND, RJ45.4
- new net HP5: ADRUINO-NANO.D2, IO2.5
- new net HP6: ADRUINO-NANO.D3, IO2.6
- new net HP7: ADRUINO-NANO.D4, IO2.7
- new net N$6: 8V-O.1, RJ45.7, RJ45.8
- net +5V: now also IO1.4; no longer DVR5V.1
- net +5VFTDI: no longer FTDI.4
- net DTR: no longer FTDI.1
- net GND: no longer -OUT.1, ADRUINO-NANO.GND, DVRGND.1, FTDI.5, FTDI.6, G.1, MINIMOSD.IGND
- net GPSRX: no longer FTDI.3
- net GPSTX: no longer FTDI.2
- net N$14: now also IO1.2, IO3.2; no longer DVRVOUT.1, VDVR.1
- net N$15: now also IO3.3, RJ45.3; no longer VMAIN.1
- net N$2: now also IO2.4; no longer 5V.1
- net N$3: now also ADRUINO-NANO.A0, R1.1, R2.2; no longer ADRUINO-NANO.A5, SCL.1
- net N$4: now also ADRUINO-NANO.D5, IO1.7; no longer ADRUINO-NANO.A4, SDA.1
- net N$5: now also V-IN.1; no longer VCC-IN.1
- net N$7: now also GND.1, RJ45.2; no longer ADRUINO-NANO.D2, K1.1
- net N$8: now also ADRUINO-NANO.D6, IO1.6; no longer ADRUINO-NANO.D3, K2.1
- net N$9: now also ADRUINO-NANO.D7, IO1.5; no longer ADRUINO-NANO.D4, K3.1
- net VIDIN: now also IO1.1; no longer DVRVIN.1
- net VIDOUT: now also IO3.4; no longer VMOD.1
Routing:
- removed copper zone on layer 1, net N$13
Other:
- board text added: "+8V"
- board text added: "-8V"
- board text added: "5V"
- board text added: "5v"
- board text added: "D2"
- board text added: "D3"
- board text added: "D4"
- board text added: "D5"
- board text added: "D6"
- board text added: "D7"
- board text added: "From switch"
- board text added: "G"
- board text added: "POCKET-GROUNDSTATION | PCB1 | REV1"
- board text added: "SCL"
- board text added: "SDA"
- board text added: "To switch"
- board text added: "Vdvr"
- board text added: "Vin"
- board text added: "Vmain"
- board text added: "Vosd"
- board text added: "Vout"
- board text removed: "Arduino NANO"
