File: eagle/PCB/PCB 1b.brd (EAGLE design)
At the start: 45 x 75 mm, 22 parts

Commit message: More PCB work
Parts:
- removed ADRUINO-NANO: NANOB, Arduino-clone:NANO
- removed GND-IN: (no value), wirepad:2,54/1,1
- removed IO2: (no value), con-lstb:MA07-1
- added ARD-SERVICE, OSD-SERVICE: EM406, SparkFun-Connectors:1X06-1MM
- added BT-BRIDGE: (no value), SparkFun-Connectors:1X03
- added G: (no value), wirepad:2,54/1,1
- added J3: (no value), SparkFun-Connectors:1X02
- added OLED: (no value), SparkFun-Connectors:1X04
- D1: value ES2D -> GF1; device diode:SMB -> diode:SMA-DO214AC
- moved U$1 63.3 mm to (26.7, 49.5)
- moved D1 12.5 mm to (35.6, 58.4), turned to 0 degrees
- moved RJ45 1.27 mm to (14.0, 5.08)
- moved V-IN 1.27 mm to (16.5, 72.4)
- turned GND to 0 degrees
- renumbered 8V-O to 8V, IO1 to DVR/MODULE-IO, IO3 to V-IO
Connections:
- net N$14 renamed DVRVIDEO-IN
- net N$15 renamed VSIGNAL-A-SW
- net VIDIN renamed RAWVIDEO_MODULE
- net VIDOUT renamed OSDSIGNAL
- removed net HP3: -OUT.1, 3.5MM.1, ADRUINO-NANO.GND, BUZZ.-, DVR/MODULE-IO.3, IO2.3, MINIMOSD.IGND, RJ45.4, V-IO.1
- removed net HP7: ADRUINO-NANO.D4, IO2.7
- removed net N$3: ADRUINO-NANO.D5, DVR/MODULE-IO.7
- removed net N$8: ADRUINO-NANO.D6, DVR/MODULE-IO.6
- removed net N$9: ADRUINO-NANO.D7, DVR/MODULE-IO.5
- new net D5: DVR/MODULE-IO.7, U$1.D5
- new net D6: DVR/MODULE-IO.6, U$1.D6
- new net D7: DVR/MODULE-IO.5, U$1.D7
- new net GROUND: -OUT.1, 3.5MM.1, BUZZ.-, DVR/MODULE-IO.3, MINIMOSD.IGND, OLED.3, RJ45.4, U$1.GND, V-IO.1
- new net N$13: J3.2, MINIMOSD.RX, OSD-SERVICE.3
- new net N$16: ARD-SERVICE.1, U$1.DTR
- new net N$18: ARD-SERVICE.2, U$1.TX0-1
- new net N$19: ARD-SERVICE.3, U$1.RX1-1
- new net N$20: ARD-SERVICE.4, U$1.VCC1
- new net N$21: ARD-SERVICE.5, U$1.GND3
- new net N$22: ARD-SERVICE.6, U$1.GND2
- new net N$4: D1.K, U$1.RAW
- net +5VFTDI: now also OSD-SERVICE.4
- net DTR: now also OSD-SERVICE.1
- net GND: now also OSD-SERVICE.5, OSD-SERVICE.6
- net GPSRX: now also J3.1, U$1.D11; no longer ADRUINO-NANO.D11, MINIMOSD.RX
- net GPSTX: now also OSD-SERVICE.2
- net HP1: now also OLED.1, U$1.A4; no longer ADRUINO-NANO.A4, IO2.1
- net HP2: now also OLED.2, U$1.A5; no longer ADRUINO-NANO.A5, IO2.2
- net HP5: now also BT-BRIDGE.3, U$1.D2; no longer ADRUINO-NANO.D2, IO2.5
- net HP6: now also BT-BRIDGE.1, U$1.D4; no longer ADRUINO-NANO.D3, IO2.6
- net N$1: now also BT-BRIDGE.2, U$1.D3; no longer ADRUINO-NANO.RAW, D1.C
- net N$10: now also U$1.D9; no longer ADRUINO-NANO.D9
- net N$11: now also G.1; no longer GND-IN.1
- net N$12: now also U$1.A0; no longer ADRUINO-NANO.A0
- net N$2: now also OLED.4, U$1.VCC; no longer ADRUINO-NANO.5V, IO2.4
Other:
- board text added: "V to DVR"
- board text removed: "Vin"
