File: eagle/PCB/PCB 1b.brd (EAGLE design)
At the start: 45 x 75 mm, 25 parts

Commit message: PCB Work
Parts:
- added AUD, SER: (no value), SparkFun-Connectors:1X01
- added J1: 0446200001, con-molex:0446200001
- added J2: AUDIO_JACK_3.5MM_KIT, SparkFun-Connectors:AUDIO-JACK-KIT
- added U$2: (no value), holes:3,0
- added X2: 0446200002, con-molex:0446200002
- BUZZ: value F/CM12P -> BUZZER-PTH; device buzzer:F/CM12P -> SparkFun-Electromechanical:BUZZER-12MM
- moved V-IO 7.62 mm to (40.6, 15.2)
- moved DVR/MODULE-IO 2.54 mm to (40.6, 30.5)
Connections:
- net N$6 renamed 8VG
- net N$7 renamed 8V
- new net AUD: 3.5MM.3, 3.5MM.4, AUD.1, RJ45.5

Commit message: Update PCB components
Parts:
- removed 3.5MM: 1503_10, con-lumberg:1503_10
- removed J1: 0446200001, con-molex:0446200001
- removed J2: AUDIO_JACK_3.5MM_KIT, SparkFun-Connectors:AUDIO-JACK-KIT
- removed X2: 0446200002, con-molex:0446200002
- added MOLEX_0446200001: 0446200001, con-molex:0446200001
- added PJ-320D: AUDIO_JACK_TRRSSMD_RA, SparkFun-Connectors:AUDIO_JACK_3.5MM_TRRS_SMD_RA
- added RJ45_MOLEX_0446200002: 0446200002, con-molex:0446200002
- moved RJ45 35.9 mm to (-21.6, 0.00)
- moved GND 1.27 mm to (8.89, 20.3), flipped to the bottom
- moved J3 1.27 mm to (10.2, 35.6)
- moved U$2 1.27 mm to (57.1, 5.08)
- flipped 8V to the bottom
- flipped AUD to the bottom, turned to 270 degrees
- flipped SER to the bottom, turned to 270 degrees
- renumbered DC-JACK to DC-005
Connections:
- removed net 8V: GND.1, RJ45.2
- removed net 8VG: 8V.1, RJ45.7, RJ45.8
- removed net AUD: 3.5MM.3, 3.5MM.4, AUD.1, RJ45.5
- removed net GROUND: -OUT.1, 3.5MM.1, BUZZ.-, DVR/MODULE-IO.3, MINIMOSD.IGND, OLED.3, RJ45.4, U$1.GND, V-IO.1
- removed net N$11: -IN.1, DC-005.1, G.1, R2.1
- removed net VSIGNAL-A-SW: 3.5MM.2, RJ45.3, V-IO.3
- new net GND1: MINIMOSD.GND1
- new net GND2: MINIMOSD.GND2
- new net N$3: AUD.1, PJ-320D.RING1, PJ-320D.TIP
- new net N$6: PJ-320D.EARTH, V-IO.3
- net GND: now also -IN.1, -OUT.1, BUZZ.-, DC-005.2, DC-005.3, DVR/MODULE-IO.3, G.1, GND.1, MINIMOSD.IGND, MINIMOSD.VGND2, OLED.3, PJ-320D.RING2, R2.1, U$1.GND, V-IO.1; no longer MINIMOSD.GND1, MINIMOSD.GND2
- net N$5: now also DC-005.1; no longer DC-005.2, DC-005.3
Routing:
- net GND: track 0.00 -> 1.32 mm
Other:
- board text added: "VIN/DVR"
- board text removed: "-8V"
- board text removed: "V to DVR"

Commit message: PCB updates
Parts:
- removed RJ45: GLX-S-88M, con-kycon:GLX-S-88M
- removed RJ45_MOLEX_0446200002: 0446200002, con-molex:0446200002
- removed U$2: (no value), holes:3,0
- BT-BRIDGE: device SparkFun-Connectors:1X03 -> SparkFun-Connectors:1X04
- moved BT-BRIDGE 1.27 mm to (24.1, 72.4)
- moved MOLEX_0446200001 0.43 mm to (14.1, 2.95)
- turned 8V to 180 degrees
- renumbered R1 to R1-18K, R2 to R2-4.7K
Connections:
- new net N$7: BT-BRIDGE.4, U$1.D13
Other:
- board text added: "D13"

Commit message: small PCB updates
Parts:
- removed +IN, -IN: (no value), wirepad:SMD1,27-2,54
- added IN+, IN-: TPTP20SQ, testpad:TP20SQ
- +5V, -OUT: value (none) -> TPTP20SQ; device wirepad:SMD1,27-2,54 -> testpad:TP20SQ
- turned +5V to 0 degrees
- turned -OUT to 180 degrees
Connections:
- net N$5 renamed +
- removed net N$17: +IN.1, R1-18K.2, VCC-O.1
- new net VCC: IN+.TP, R1-18K.2, VCC-O.1
- net +5V: now also +5V.TP; no longer +5V.1
- net GND: now also -OUT.TP, IN-.TP; no longer -IN.1, -OUT.1
Changed lines of the file:
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@@
 <attribute name="MF" value="" x="8.89" y="66.04" size="1.778" layer="27" rot="R180" display="off"/>
 <attribute name="MPN" value="" x="8.89" y="66.04" size="1.778" layer="27" rot="R180" display="off"/>
-<attribute name="NAME" x="12.7" y="67.31" size="1.27" layer="25" rot="R180"/>
+<attribute name="NAME" x="11.43" y="72.39" size="1.27" layer="25" rot="R180"/>
 <attribute name="OC_FARNELL" value="unknown" x="8.89" y="66.04" size="1.778" layer="27" rot="R180" display="off"/>
 <attribute name="OC_NEWARK" value="unknown" x="8.89" y="66.04" size="1.778" layer="27" rot="R180" display="off"/>
@@
 </element>
 <element name="MINIMOSD" library="FPVTools" package="MMOSDNVDVID" value="MICROMINIMOSDPWR" x="21.59" y="25.4" rot="R180"/>
-<element name="-IN" library="wirepad" library_urn="urn:adsk.eagle:library:412" package="SMD1,27-2,54" package3d_urn="urn:adsk.eagle:package:30839/1" value="" x="15.24" y="68.58" smashed="yes" rot="R90">
-<attribute name="NAME" x="18.91" y="66.51" size="1.27" layer="25" rot="R180"/>
-<attribute name="VALUE" x="15.24" y="68.58" size="0.0254" layer="27" rot="R90"/>
-</element>
-<element name="-OUT" library="wirepad" library_urn="urn:adsk.eagle:library:412" package="SMD1,27-2,54" package3d_urn="urn:adsk.eagle:package:30839/1" value="" x="29.21" y="68.58" smashed="yes" rot="R90">
-<attribute name="NAME" x="27.8" y="66.51" size="1.27" layer="25" rot="R180"/>
-<attribute name="VALUE" x="29.21" y="68.58" size="0.0254" layer="27" rot="R90"/>
-</element>
-<element name="+5V" library="wirepad" library_urn="urn:adsk.eagle:library:412" package="SMD1,27-2,54" package3d_urn="urn:adsk.eagle:package:30839/1" value="" x="29.21" y="58.42" smashed="yes" rot="R90">
-<attribute name="NAME" x="27.8" y="61.43" size="1.27" layer="25" rot="R180"/>
-<attribute name="VALUE" x="29.21" y="58.42" size="0.0254" layer="27" rot="R90"/>
-</element>
-<element name="+IN" library="wirepad" library_urn="urn:adsk.eagle:library:412" package="SMD1,27-2,54" package3d_urn="urn:adsk.eagle:package:30839/1" value="" x="15.24" y="58.42" smashed="yes" rot="R270">
-<attribute name="NAME" x="19.19" y="61.76" size="1.27" layer="25" rot="R180"/>
-<attribute name="VALUE" x="15.24" y="58.42" size="0.0254" layer="27" rot="R270"/>
-</element>
 <element name="R1-18K" library="rcl" library_urn="urn:adsk.eagle:library:334" package="M1206" package3d_urn="urn:adsk.eagle:package:23566/1" value="18k Ohm" x="11.43" y="49.53" smashed="yes" rot="R180">
 <attribute name="NAME" x="13.97" y="46.99" size="1.27" layer="25" rot="R180"/>
@@
 <attribute name="SF_ID" value="PRT-12639" x="30.48" y="0" size="1.778" layer="27" rot="R90" display="off"/>
 </element>
+<element name="IN-" library="testpad" library_urn="urn:adsk.eagle:library:385" package="TP20SQ" package3d_urn="urn:adsk.eagle:package:27980/1" value="TPTP20SQ" x="15.24" y="68.58" rot="R180">
+<attribute name="TP_SIGNAL_NAME" value="" x="15.24" y="68.58" size="1.778" layer="27" rot="R180" display="off"/>
+</element>
+<element name="IN+" library="testpad" library_urn="urn:adsk.eagle:library:385" package="TP20SQ" package3d_urn="urn:adsk.eagle:package:27980/1" value="TPTP20SQ" x="15.24" y="58.42">
+<attribute name="TP_SIGNAL_NAME" value="" x="15.24" y="58.42" size="1.778" layer="27" display="off"/>
+</element>
+<element name="+5V" library="testpad" library_urn="urn:adsk.eagle:library:385" package="TP20SQ" package3d_urn="urn:adsk.eagle:package:27980/1" value="TPTP20SQ" x="29.21" y="58.42">
+<attribute name="TP_SIGNAL_NAME" value="" x="29.21" y="58.42" size="1.778" layer="27" display="off"/>
+</element>
+<element name="-OUT" library="testpad" library_urn="urn:adsk.eagle:library:385" package="TP20SQ" package3d_urn="urn:adsk.eagle:package:27980/1" value="TPTP20SQ" x="29.21" y="68.58" rot="R180">
+<attribute name="TP_SIGNAL_NAME" value="" x="29.21" y="68.58" size="1.778" layer="27" rot="R180" display="off"/>
+</element>
 </elements>
 <signals>
@@
 <wire x1="2.54" y1="22.86" x2="21.59" y2="43.18" width="0" layer="19" extent="1-1"/>
 </signal>
-<signal name="N$5">
+<signal name="+">
 <contactref element="V-IN" pad="1"/>
 <contactref element="DC-005" pad="1"/>
@@
 <signal name="+5V">
 <contactref element="MINIMOSD" pad="IVCC"/>
-<contactref element="+5V" pad="1"/>
 <contactref element="DVR/MODULE-IO" pad="4"/>
 <contactref element="D1" pad="A"/>
+<contactref element="+5V" pad="TP"/>
 <wire x1="29.21" y1="58.42" x2="33.51" y2="58.42" width="0" layer="19" extent="1-1"/>
 <wire x1="21.59" y1="34.33" x2="29.21" y2="58.42" width="0" layer="19" extent="1-1"/>
@@
 </signal>
 <signal name="GND">
-<contactref element="-IN" pad="1"/>
 <contactref element="G" pad="1"/>
 <contactref element="MINIMOSD" pad="IGND"/>
-<contactref element="-OUT" pad="1"/>
 <contactref element="DVR/MODULE-IO" pad="3"/>
 <contactref element="BUZZ" pad="-"/>
 <contactref element="U$1" pad="GND"/>
-<wire x1="14.9225" y1="68.58" x2="15.24" y2="68.58" width="0.762" layer="1"/>
 <contactref element="OLED" pad="3"/>
 <contactref element="GND" pad="1"/>
@@
 <wire x1="5.08" y1="30.29" x2="5.08" y2="29.29" width="0.381" layer="1"/>
 <contactref element="PJ-320D" pad="RING2"/>
+<contactref element="IN-" pad="TP"/>
+<contactref element="-OUT" pad="TP"/>
 <wire x1="29.21" y1="68.58" x2="38.1" y2="70.56" width="0" layer="19" extent="1-1"/>
 <wire x1="20.32" y1="72.39" x2="29.21" y2="68.58" width="0" layer="19" extent="1-1"/>
 <wire x1="15.24" y1="68.58" x2="20.32" y2="72.39" width="0" layer="19" extent="1-1"/>
-<wire x1="8.89" y1="69.04" x2="14.9225" y2="68.58" width="0" layer="19" extent="1-1"/>
+<wire x1="8.89" y1="69.04" x2="15.24" y2="68.58" width="0" layer="19" extent="1-1"/>
 <wire x1="4.09" y1="66.04" x2="8.89" y2="69.04" width="0" layer="19" extent="1-1"/>
 <wire x1="25.53" y1="49.53" x2="29.21" y2="68.58" width="0" layer="19" extent="1-1"/>
@@
 <wire x1="40.64" y1="13.97" x2="40.64" y2="25.4" width="0" layer="19" extent="1-1"/>
 </signal>
-<signal name="N$17">
+<signal name="VCC">
 <contactref element="R1-18K" pad="2"/>
-<contactref element="+IN" pad="1"/>
 <contactref element="VCC-O" pad="1"/>
+<contactref element="IN+" pad="TP"/>
 <wire x1="7.62" y1="59.69" x2="15.24" y2="58.42" width="0" layer="19" extent="1-1"/>
 <wire x1="10.03" y1="49.53" x2="15.24" y2="58.42" width="0" layer="19" extent="1-1"/>

Commit message: PCB updates
Parts:
- moved J3 7.73 mm to (8.89, 27.9)
- moved OSD-SERVICE 1.27 mm to (3.81, 33.0)
Connections:
- removed net GND1: MINIMOSD.GND1
- removed net GND2: MINIMOSD.GND2
- removed net N$20: ARD-SERVICE.4, U$1.VCC1
- removed net N$6: PJ-320D.EARTH, V-IO.3
- new net 8V: 8V.1, MOLEX_0446200001.7, MOLEX_0446200001.8
- new net AUDIO: AUD.1, MOLEX_0446200001.5, PJ-320D.RING1, PJ-320D.TIP
- new net N$5: MINIMOSD.GND2, OSD-SERVICE.1
- new net V: ARD-SERVICE.4, U$1.RX01
- new net VMAIN: MOLEX_0446200001.3, PJ-320D.EARTH, V-IO.3
- net +5VFTDI: now also OSD-SERVICE.3; no longer OSD-SERVICE.4
- net DTR: now also OSD-SERVICE.6; no longer OSD-SERVICE.1
- net GND: now also MOLEX_0446200001.2, MOLEX_0446200001.4; no longer OSD-SERVICE.5, OSD-SERVICE.6
- net GPSTX: now also OSD-SERVICE.5; no longer OSD-SERVICE.2
- net N$16: now also U$1.BLK; no longer U$1.DTR
- net N$18: now also U$1.G; no longer U$1.TX0-1
- net N$19: now also U$1.5V; no longer U$1.RX1-1
- net N$21: now also U$1.TX01; no longer U$1.GND3
- net N$22: now also U$1.DTR; no longer U$1.GND2
- net N$3: now also MINIMOSD.GND1, OSD-SERVICE.2; no longer AUD.1, PJ-320D.RING1, PJ-320D.TIP
- net RX: now also OSD-SERVICE.4; no longer OSD-SERVICE.3
Routing:
- net N$3: track 0.00 -> 12.6 mm
- net N$5: track 0.00 -> 10.5 mm
- net GND: track 1.00 -> 0.00 mm

Commit message: More PCB work
Parts:
- moved +5V 1.27 mm to (30.5, 58.4)
- moved -OUT 1.27 mm to (30.5, 68.6)
- moved D1 1.27 mm to (36.8, 58.4)
Changed lines of the file:
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@@
 <layer number="20" name="Dimension" color="24" fill="1" visible="yes" active="yes"/>
 <layer number="21" name="tPlace" color="7" fill="1" visible="yes" active="yes"/>
-<layer number="22" name="bPlace" color="7" fill="1" visible="no" active="yes"/>
+<layer number="22" name="bPlace" color="7" fill="1" visible="yes" active="yes"/>
 <layer number="23" name="tOrigins" color="15" fill="1" visible="yes" active="yes"/>
-<layer number="24" name="bOrigins" color="15" fill="1" visible="no" active="yes"/>
+<layer number="24" name="bOrigins" color="15" fill="1" visible="yes" active="yes"/>
 <layer number="25" name="tNames" color="7" fill="1" visible="yes" active="yes"/>
-<layer number="26" name="bNames" color="7" fill="1" visible="no" active="yes"/>
+<layer number="26" name="bNames" color="7" fill="1" visible="yes" active="yes"/>
 <layer number="27" name="tValues" color="7" fill="1" visible="no" active="yes"/>
 <layer number="28" name="bValues" color="7" fill="1" visible="no" active="yes"/>
@@
 <layer number="38" name="bTest" color="7" fill="1" visible="no" active="yes"/>
 <layer number="39" name="tKeepout" color="4" fill="11" visible="yes" active="yes"/>
-<layer number="40" name="bKeepout" color="1" fill="11" visible="no" active="yes"/>
+<layer number="40" name="bKeepout" color="1" fill="11" visible="yes" active="yes"/>
 <layer number="41" name="tRestrict" color="4" fill="10" visible="yes" active="yes"/>
-<layer number="42" name="bRestrict" color="1" fill="10" visible="no" active="yes"/>
+<layer number="42" name="bRestrict" color="1" fill="10" visible="yes" active="yes"/>
 <layer number="43" name="vRestrict" color="2" fill="10" visible="no" active="yes"/>
 <layer number="44" name="Drills" color="7" fill="1" visible="no" active="yes"/>
@@
 <layer number="50" name="dxf" color="7" fill="1" visible="no" active="no"/>
 <layer number="51" name="tDocu" color="7" fill="1" visible="yes" active="yes"/>
-<layer number="52" name="bDocu" color="7" fill="1" visible="no" active="yes"/>
+<layer number="52" name="bDocu" color="7" fill="1" visible="yes" active="yes"/>
 <layer number="53" name="tGND_GNDA" color="7" fill="9" visible="no" active="no"/>
 <layer number="54" name="bGND_GNDA" color="1" fill="9" visible="no" active="no"/>
@@
 <attribute name="PROD_ID" value="CONN-09696" x="2.54" y="22.86" size="1.778" layer="27" rot="R270" display="off"/>
 </element>
-<element name="D1" library="diode" library_urn="urn:adsk.eagle:library:210" package="SMA-DO214AC" package3d_urn="urn:adsk.eagle:package:43452/2" value="GF1" x="35.56" y="58.42"/>
+<element name="D1" library="diode" library_urn="urn:adsk.eagle:library:210" package="SMA-DO214AC" package3d_urn="urn:adsk.eagle:package:43452/2" value="GF1" x="36.83" y="58.42"/>
 <element name="J3" library="SparkFun-Connectors" library_urn="urn:adsk.eagle:library:513" package="1X02" package3d_urn="urn:adsk.eagle:package:38039/1" value="" x="8.89" y="27.94" rot="R270"/>
 <element name="ARD-SERVICE" library="SparkFun-Connectors" library_urn="urn:adsk.eagle:library:513" package="1X06-1MM" package3d_urn="urn:adsk.eagle:package:38023/1" value="EM406" x="41.91" y="46.99" smashed="yes" rot="R90">
@@
 <attribute name="TP_SIGNAL_NAME" value="" x="15.24" y="58.42" size="1.778" layer="27" display="off"/>
 </element>
-<element name="+5V" library="testpad" library_urn="urn:adsk.eagle:library:385" package="TP20SQ" package3d_urn="urn:adsk.eagle:package:27980/1" value="TPTP20SQ" x="29.21" y="58.42">
-<attribute name="TP_SIGNAL_NAME" value="" x="29.21" y="58.42" size="1.778" layer="27" display="off"/>
+<element name="+5V" library="testpad" library_urn="urn:adsk.eagle:library:385" package="TP20SQ" package3d_urn="urn:adsk.eagle:package:27980/1" value="TPTP20SQ" x="30.48" y="58.42">
+<attribute name="TP_SIGNAL_NAME" value="" x="30.48" y="58.42" size="1.778" layer="27" display="off"/>
 </element>
-<element name="-OUT" library="testpad" library_urn="urn:adsk.eagle:library:385" package="TP20SQ" package3d_urn="urn:adsk.eagle:package:27980/1" value="TPTP20SQ" x="29.21" y="68.58" rot="R180">
-<attribute name="TP_SIGNAL_NAME" value="" x="29.21" y="68.58" size="1.778" layer="27" rot="R180" display="off"/>
+<element name="-OUT" library="testpad" library_urn="urn:adsk.eagle:library:385" package="TP20SQ" package3d_urn="urn:adsk.eagle:package:27980/1" value="TPTP20SQ" x="30.48" y="68.58" rot="R180">
+<attribute name="TP_SIGNAL_NAME" value="" x="30.48" y="68.58" size="1.778" layer="27" rot="R180" display="off"/>
 </element>
 </elements>
@@
 <contactref element="D1" pad="A"/>
 <contactref element="+5V" pad="TP"/>
-<wire x1="29.21" y1="58.42" x2="33.51" y2="58.42" width="0" layer="19" extent="1-1"/>
-<wire x1="21.59" y1="34.33" x2="29.21" y2="58.42" width="0" layer="19" extent="1-1"/>
+<wire x1="30.48" y1="58.42" x2="34.78" y2="58.42" width="0" layer="19" extent="1-1"/>
+<wire x1="21.59" y1="34.33" x2="30.48" y2="58.42" width="0" layer="19" extent="1-1"/>
 <wire x1="40.64" y1="30.48" x2="21.59" y2="34.33" width="0" layer="19" extent="1-1"/>
 </signal>
@@
 <contactref element="MOLEX_0446200001" pad="4"/>
 <contactref element="MOLEX_0446200001" pad="2"/>
-<wire x1="29.21" y1="68.58" x2="38.1" y2="70.56" width="0" layer="19" extent="1-1"/>
-<wire x1="20.32" y1="72.39" x2="29.21" y2="68.58" width="0" layer="19" extent="1-1"/>
+<wire x1="30.48" y1="68.58" x2="38.1" y2="70.56" width="0" layer="19" extent="1-1"/>
+<wire x1="20.32" y1="72.39" x2="30.48" y2="68.58" width="0" layer="19" extent="1-1"/>
 <wire x1="15.24" y1="68.58" x2="20.32" y2="72.39" width="0" layer="19" extent="1-1"/>
 <wire x1="8.89" y1="69.04" x2="15.24" y2="68.58" width="0" layer="19" extent="1-1"/>
 <wire x1="4.09" y1="66.04" x2="8.89" y2="69.04" width="0" layer="19" extent="1-1"/>
-<wire x1="25.53" y1="49.53" x2="29.21" y2="68.58" width="0" layer="19" extent="1-1"/>
+<wire x1="25.53" y1="49.53" x2="30.48" y2="68.58" width="0" layer="19" extent="1-1"/>
 <wire x1="30.48" y1="39.37" x2="25.53" y2="49.53" width="0" layer="19" extent="1-1"/>
 <wire x1="19.05" y1="34.33" x2="30.48" y2="39.37" width="0" layer="19" extent="1-1"/>
@@
 <contactref element="U$1" pad="RAW"/>
 <contactref element="D1" pad="K"/>
-<wire x1="33.02" y1="39.37" x2="37.61" y2="58.42" width="0" layer="19" extent="1-1"/>
+<wire x1="33.02" y1="39.37" x2="38.88" y2="58.42" width="0" layer="19" extent="1-1"/>
 </signal>
 <signal name="RX" class="1">
