File: eagle/PCB/PCB 1b.sch (EAGLE design)
At the start: 29 parts

Commit message: PCB updates
Parts:
- removed RJ45: GLX-S-88M, con-kycon:GLX-S-88M
- removed RJ45_MOLEX_0446200002: 0446200002, con-molex:0446200002
- BT-BRIDGE: device SparkFun-Connectors:CONN_03 -> SparkFun-Connectors:CONN_04
- renumbered R1 to R1-18K, R2 to R2-4.7K
Connections:
- new net N$7: BT-BRIDGE.4, U$1.D13
Other:
- note added: "D13"
Changed lines of the file:
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@@
 </classes>
 <parts>
-<part name="RJ45" library="con-kycon" library_urn="urn:adsk.eagle:library:157" deviceset="GLX-S-88M" device="" package3d_urn="urn:adsk.eagle:package:7680/1"/>
 <part name="BUZZ" library="SparkFun-Electromechanical" library_urn="urn:adsk.eagle:library:516" deviceset="BUZZER" device="-PTH" package3d_urn="urn:adsk.eagle:package:38558/1">
 <attribute name="SPICEPREFIX" value="X"/>
@@
 <part name="+5V" library="wirepad" library_urn="urn:adsk.eagle:library:412" deviceset="SMD2" device="" package3d_urn="urn:adsk.eagle:package:30839/1"/>
 <part name="+IN" library="wirepad" library_urn="urn:adsk.eagle:library:412" deviceset="SMD2" device="" package3d_urn="urn:adsk.eagle:package:30839/1"/>
-<part name="R1" library="rcl" library_urn="urn:adsk.eagle:library:334" deviceset="R-EU_" device="M1206" package3d_urn="urn:adsk.eagle:package:23566/1" value="18k Ohm"/>
-<part name="R2" library="rcl" library_urn="urn:adsk.eagle:library:334" deviceset="R-EU_" device="M1206" package3d_urn="urn:adsk.eagle:package:23566/1" value="4.7 kOhm"/>
+<part name="R1-18K" library="rcl" library_urn="urn:adsk.eagle:library:334" deviceset="R-EU_" device="M1206" package3d_urn="urn:adsk.eagle:package:23566/1" value="18k Ohm"/>
+<part name="R2-4.7K" library="rcl" library_urn="urn:adsk.eagle:library:334" deviceset="R-EU_" device="M1206" package3d_urn="urn:adsk.eagle:package:23566/1" value="4.7 kOhm"/>
 <part name="8V" library="wirepad" library_urn="urn:adsk.eagle:library:412" deviceset="2,54/1,1" device="" package3d_urn="urn:adsk.eagle:package:30836/1"/>
 <part name="GND" library="wirepad" library_urn="urn:adsk.eagle:library:412" deviceset="2,54/1,1" device="" package3d_urn="urn:adsk.eagle:package:30836/1"/>
@@
 <part name="V-IO" library="con-lstb" library_urn="urn:adsk.eagle:library:162" deviceset="MA04-1" device="" package3d_urn="urn:adsk.eagle:package:8337/1"/>
 <part name="U$1" library="Arduino-clone" deviceset="ABK-PRO-MINI" device=""/>
-<part name="BT-BRIDGE" library="SparkFun-Connectors" library_urn="urn:adsk.eagle:library:513" deviceset="CONN_03" device="" package3d_urn="urn:adsk.eagle:package:38063/1"/>
+<part name="BT-BRIDGE" library="SparkFun-Connectors" library_urn="urn:adsk.eagle:library:513" deviceset="CONN_04" device="" package3d_urn="urn:adsk.eagle:package:38085/1"/>
 <part name="OLED" library="SparkFun-Connectors" library_urn="urn:adsk.eagle:library:513" deviceset="CONN_04" device="" package3d_urn="urn:adsk.eagle:package:38085/1"/>
 <part name="D1" library="diode" library_urn="urn:adsk.eagle:library:210" deviceset="GF1" device="" package3d_urn="urn:adsk.eagle:package:43452/2"/>
@@
 <part name="SER" library="SparkFun-Connectors" library_urn="urn:adsk.eagle:library:513" deviceset="CONN_01" device="" package3d_urn="urn:adsk.eagle:package:38028/1"/>
 <part name="AUD" library="SparkFun-Connectors" library_urn="urn:adsk.eagle:library:513" deviceset="CONN_01" device="" package3d_urn="urn:adsk.eagle:package:38028/1"/>
-<part name="RJ45_MOLEX_0446200002" library="con-molex" library_urn="urn:adsk.eagle:library:165" deviceset="0446200002" device=""/>
 <part name="MOLEX_0446200001" library="con-molex" library_urn="urn:adsk.eagle:library:165" deviceset="0446200001" device="" value="0446200001"/>
 <part name="PJ-320D" library="SparkFun-Connectors" library_urn="urn:adsk.eagle:library:513" deviceset="AUDIO_JACK_TRRS" device="SMD_RA" package3d_urn="urn:adsk.eagle:package:38268/1"/>
@@
 <text x="65.532" y="105.918" size="1.778" layer="91">5:AUD
 </text>
+<text x="210.82" y="195.58" size="1.778" layer="91" rot="R90">D13</text>
 </plain>
 <instances>
-<instance part="RJ45" gate="G$1" x="86.36" y="106.68" rot="R180"/>
 <instance part="BUZZ" gate="G$1" x="238.76" y="93.98" smashed="yes">
 <attribute name="VALUE" x="233.68" y="83.82" size="1.778" layer="96"/>
@@
 <instance part="+5V" gate="1" x="292.1" y="83.82" rot="R270"/>
 <instance part="+IN" gate="1" x="292.1" y="99.06" rot="R90"/>
-<instance part="R1" gate="G$1" x="317.5" y="93.98" rot="R90"/>
-<instance part="R2" gate="G$1" x="317.5" y="76.2" rot="R90"/>
+<instance part="R1-18K" gate="G$1" x="317.5" y="93.98" rot="R90"/>
+<instance part="R2-4.7K" gate="G$1" x="317.5" y="76.2" rot="R90"/>
 <instance part="8V" gate="1" x="76.2" y="165.1" rot="R270"/>
 <instance part="GND" gate="1" x="68.58" y="165.1" rot="R270"/>
@@
 </instance>
 <instance part="U$1" gate="G$1" x="177.8" y="101.6" rot="R180"/>
-<instance part="BT-BRIDGE" gate="J$1" x="205.74" y="190.5" rot="R270"/>
+<instance part="BT-BRIDGE" gate="G$1" x="205.74" y="190.5" rot="R270"/>
 <instance part="OLED" gate="G$1" x="96.52" y="193.04" rot="R270"/>
 <instance part="D1" gate="D" x="165.1" y="63.5" rot="R180"/>
@@
 <instance part="SER" gate="G$1" x="226.06" y="175.26" rot="R90"/>
 <instance part="AUD" gate="G$1" x="104.14" y="50.8" rot="R90"/>
-<instance part="RJ45_MOLEX_0446200002" gate="P" x="157.48" y="276.86"/>
 <instance part="MOLEX_0446200001" gate="P" x="96.52" y="246.38"/>
 <instance part="PJ-320D" gate="G$1" x="78.74" y="35.56"/>
@@
 <wire x1="330.2" y1="96.52" x2="330.2" y2="99.06" width="0.1524" layer="91"/>
 <junction x="330.2" y="96.52"/>
-<pinref part="R2" gate="G$1" pin="1"/>
+<pinref part="R2-4.7K" gate="G$1" pin="1"/>
 <wire x1="317.5" y1="71.12" x2="317.5" y2="68.58" width="0.1524" layer="91"/>
 <wire x1="317.5" y1="68.58" x2="325.12" y2="68.58" width="0.1524" layer="91"/>
@@
 <pinref part="U$1" gate="G$1" pin="D2"/>
 <wire x1="208.28" y1="99.06" x2="200.66" y2="99.06" width="0.1524" layer="91"/>
-<pinref part="BT-BRIDGE" gate="J$1" pin="3"/>
-<wire x1="208.28" y1="182.88" x2="208.28" y2="99.06" width="0.1524" layer="91"/>
+<pinref part="BT-BRIDGE" gate="G$1" pin="3"/>
+<wire x1="208.28" y1="185.42" x2="208.28" y2="99.06" width="0.1524" layer="91"/>
 </segment>
 </net>
 <net name="HP6" class="1">
 <segment>
-<pinref part="BT-BRIDGE" gate="J$1" pin="1"/>
+<pinref part="BT-BRIDGE" gate="G$1" pin="1"/>
 <pinref part="U$1" gate="G$1" pin="D4"/>
 <wire x1="203.2" y1="104.14" x2="200.66" y2="104.14" width="0.1524" layer="91"/>
-<wire x1="203.2" y1="182.88" x2="203.2" y2="104.14" width="0.1524" layer="91"/>
+<wire x1="203.2" y1="185.42" x2="203.2" y2="104.14" width="0.1524" layer="91"/>
 </segment>
 </net>
@@
 <net name="N$17" class="0">
 <segment>
-<pinref part="R1" gate="G$1" pin="2"/>
+<pinref part="R1-18K" gate="G$1" pin="2"/>
 <wire x1="317.5" y1="99.06" x2="317.5" y2="127" width="0.1524" layer="91"/>
 <pinref part="+IN" gate="1" pin="P"/>
@@
 <wire x1="226.06" y1="127" x2="254" y2="91.44" width="0.1524" layer="91"/>
 <wire x1="254" y1="91.44" x2="261.62" y2="88.9" width="0.1524" layer="91"/>
-<pinref part="R1" gate="G$1" pin="1"/>
-<pinref part="R2" gate="G$1" pin="2"/>
+<pinref part="R1-18K" gate="G$1" pin="1"/>
+<pinref part="R2-4.7K" gate="G$1" pin="2"/>
 <wire x1="317.5" y1="88.9" x2="317.5" y2="81.28" width="0.1524" layer="91"/>
 <wire x1="261.62" y1="88.9" x2="317.5" y2="88.9" width="0.1524" layer="91"/>
@@
 <segment>
 <pinref part="U$1" gate="G$1" pin="D3"/>
-<pinref part="BT-BRIDGE" gate="J$1" pin="2"/>
-<wire x1="205.74" y1="182.88" x2="205.74" y2="101.6" width="0.1524" layer="91"/>
+<pinref part="BT-BRIDGE" gate="G$1" pin="2"/>
+<wire x1="205.74" y1="185.42" x2="205.74" y2="101.6" width="0.1524" layer="91"/>
 <wire x1="205.74" y1="101.6" x2="200.66" y2="101.6" width="0.1524" layer="91"/>
 </segment>
@@
 </segment>
 </net>
+<net name="N$7" class="1">
+<segment>
+<pinref part="U$1" gate="G$1" pin="D13"/>
+<wire x1="162.56" y1="109.22" x2="147.32" y2="109.22" width="0.1524" layer="91"/>
+<wire x1="147.32" y1="109.22" x2="147.32" y2="177.8" width="0.1524" layer="91"/>
+<pinref part="BT-BRIDGE" gate="G$1" pin="4"/>
+<wire x1="147.32" y1="177.8" x2="210.82" y2="177.8" width="0.1524" layer="91"/>
+<wire x1="210.82" y1="177.8" x2="210.82" y2="185.42" width="0.1524" layer="91"/>
+</segment>
+</net>

Commit message: small PCB updates
Parts:
- removed +IN, -IN: (no value), wirepad:SMD2
- added IN+, IN-: TPTP20SQ, testpad:TPTP20SQ
- +5V, -OUT: value (none) -> TPTP20SQ; device wirepad:SMD2 -> testpad:TPTP20SQ
Connections:
- net N$5 renamed +
- removed net N$17: +IN.P, R1-18K.2, VCC-O.P
- new net VCC: IN+.TP, R1-18K.2, VCC-O.P
- net +5V: now also +5V.TP; no longer +5V.P
- net GND: now also -OUT.TP, IN-.TP; no longer -IN.P, -OUT.P
Changed lines of the file:
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@@
 <part name="VCC-O" library="wirepad" library_urn="urn:adsk.eagle:library:412" deviceset="2,54/1,1" device="" package3d_urn="urn:adsk.eagle:package:30836/1"/>
 <part name="MINIMOSD" library="FPVTools" deviceset="MICROMINIMOSDPWR" device=""/>
-<part name="-IN" library="wirepad" library_urn="urn:adsk.eagle:library:412" deviceset="SMD2" device="" package3d_urn="urn:adsk.eagle:package:30839/1"/>
-<part name="-OUT" library="wirepad" library_urn="urn:adsk.eagle:library:412" deviceset="SMD2" device="" package3d_urn="urn:adsk.eagle:package:30839/1"/>
-<part name="+5V" library="wirepad" library_urn="urn:adsk.eagle:library:412" deviceset="SMD2" device="" package3d_urn="urn:adsk.eagle:package:30839/1"/>
-<part name="+IN" library="wirepad" library_urn="urn:adsk.eagle:library:412" deviceset="SMD2" device="" package3d_urn="urn:adsk.eagle:package:30839/1"/>
 <part name="R1-18K" library="rcl" library_urn="urn:adsk.eagle:library:334" deviceset="R-EU_" device="M1206" package3d_urn="urn:adsk.eagle:package:23566/1" value="18k Ohm"/>
 <part name="R2-4.7K" library="rcl" library_urn="urn:adsk.eagle:library:334" deviceset="R-EU_" device="M1206" package3d_urn="urn:adsk.eagle:package:23566/1" value="4.7 kOhm"/>
@@
 <part name="MOLEX_0446200001" library="con-molex" library_urn="urn:adsk.eagle:library:165" deviceset="0446200001" device="" value="0446200001"/>
 <part name="PJ-320D" library="SparkFun-Connectors" library_urn="urn:adsk.eagle:library:513" deviceset="AUDIO_JACK_TRRS" device="SMD_RA" package3d_urn="urn:adsk.eagle:package:38268/1"/>
+<part name="IN-" library="testpad" library_urn="urn:adsk.eagle:library:385" deviceset="TP" device="TP20SQ" package3d_urn="urn:adsk.eagle:package:27980/1"/>
+<part name="IN+" library="testpad" library_urn="urn:adsk.eagle:library:385" deviceset="TP" device="TP20SQ" package3d_urn="urn:adsk.eagle:package:27980/1"/>
+<part name="+5V" library="testpad" library_urn="urn:adsk.eagle:library:385" deviceset="TP" device="TP20SQ" package3d_urn="urn:adsk.eagle:package:27980/1"/>
+<part name="-OUT" library="testpad" library_urn="urn:adsk.eagle:library:385" deviceset="TP" device="TP20SQ" package3d_urn="urn:adsk.eagle:package:27980/1"/>
 </parts>
 <sheets>
@@
 <instance part="VCC-O" gate="1" x="330.2" y="152.4"/>
 <instance part="MINIMOSD" gate="G$1" x="256.54" y="137.16"/>
-<instance part="-IN" gate="1" x="302.26" y="99.06" rot="R90"/>
-<instance part="-OUT" gate="1" x="302.26" y="83.82" rot="R270"/>
-<instance part="+5V" gate="1" x="292.1" y="83.82" rot="R270"/>
-<instance part="+IN" gate="1" x="292.1" y="99.06" rot="R90"/>
 <instance part="R1-18K" gate="G$1" x="317.5" y="93.98" rot="R90"/>
 <instance part="R2-4.7K" gate="G$1" x="317.5" y="76.2" rot="R90"/>
@@
 <instance part="MOLEX_0446200001" gate="P" x="96.52" y="246.38"/>
 <instance part="PJ-320D" gate="G$1" x="78.74" y="35.56"/>
+<instance part="IN-" gate="G$1" x="302.26" y="99.06" rot="R180"/>
+<instance part="IN+" gate="G$1" x="292.1" y="99.06" rot="R180"/>
+<instance part="+5V" gate="G$1" x="292.1" y="83.82"/>
+<instance part="-OUT" gate="G$1" x="302.26" y="83.82"/>
 </instances>
 <busses>
@@
 </segment>
 </net>
-<net name="N$5" class="0">
+<net name="+" class="0">
 <segment>
 <pinref part="V-IN" gate="1" pin="P"/>
@@
 <pinref part="MINIMOSD" gate="G$1" pin="IVCC"/>
 <label x="251.46" y="111.76" size="1.778" layer="95" rot="R180" xref="yes"/>
-<pinref part="+5V" gate="1" pin="P"/>
 <wire x1="292.1" y1="81.28" x2="292.1" y2="73.66" width="0.1524" layer="91"/>
 <wire x1="292.1" y1="73.66" x2="292.1" y2="63.5" width="0.1524" layer="91"/>
@@
 <junction x="198.12" y="63.5"/>
 <junction x="167.64" y="63.5"/>
+<pinref part="+5V" gate="G$1" pin="TP"/>
 </segment>
 </net>
 <net name="GND" class="0">
 <segment>
-<pinref part="-IN" gate="1" pin="P"/>
-<wire x1="302.26" y1="101.6" x2="302.26" y2="116.84" width="0.1524" layer="91"/>
 <pinref part="G" gate="1" pin="P"/>
 <wire x1="322.58" y1="137.16" x2="322.58" y2="142.24" width="0.1524" layer="91"/>
@@
 <wire x1="261.62" y1="116.84" x2="261.62" y2="111.76" width="0.1524" layer="91"/>
 <label x="261.62" y="111.76" size="1.778" layer="95" xref="yes"/>
-<pinref part="-OUT" gate="1" pin="P"/>
 <wire x1="302.26" y1="81.28" x2="302.26" y2="78.74" width="0.1524" layer="91"/>
 <wire x1="302.26" y1="78.74" x2="302.26" y2="68.58" width="0.1524" layer="91"/>
@@
 <wire x1="157.48" y1="91.44" x2="162.56" y2="91.44" width="0.1524" layer="91"/>
 <pinref part="OLED" gate="G$1" pin="3"/>
-<wire x1="302.26" y1="101.6" x2="302.26" y2="78.74" width="0.1524" layer="91"/>
-<junction x="302.26" y="101.6"/>
+<wire x1="302.26" y1="116.84" x2="302.26" y2="101.6" width="0.1524" layer="91"/>
+<wire x1="302.26" y1="101.6" x2="302.26" y2="81.28" width="0.1524" layer="91"/>
+<wire x1="302.26" y1="81.28" x2="302.26" y2="78.74" width="0.1524" layer="91"/>
 <wire x1="332.74" y1="142.24" x2="342.9" y2="142.24" width="0.1524" layer="91"/>
 <junction x="332.74" y="142.24"/>
@@
 <pinref part="PJ-320D" gate="G$1" pin="RING2"/>
 <wire x1="83.82" y1="30.48" x2="129.54" y2="30.48" width="0.1524" layer="91"/>
+<pinref part="IN-" gate="G$1" pin="TP"/>
+<junction x="302.26" y="101.6"/>
+<pinref part="-OUT" gate="G$1" pin="TP"/>
+<junction x="302.26" y="81.28"/>
 </segment>
 </net>
@@
 </segment>
 </net>
-<net name="N$17" class="0">
+<net name="VCC" class="0">
 <segment>
 <pinref part="R1-18K" gate="G$1" pin="2"/>
 <wire x1="317.5" y1="99.06" x2="317.5" y2="127" width="0.1524" layer="91"/>
-<pinref part="+IN" gate="1" pin="P"/>
 <wire x1="292.1" y1="101.6" x2="317.5" y2="127" width="0.1524" layer="91"/>
 <wire x1="317.5" y1="127" x2="317.5" y2="152.4" width="0.1524" layer="91"/>
@@
 <wire x1="317.5" y1="152.4" x2="332.74" y2="152.4" width="0.1524" layer="91"/>
 <junction x="317.5" y="127"/>
-</segment>
-</net>
+<pinref part="IN+" gate="G$1" pin="TP"/>
+</segment>
+</net>

Commit message: PCB updates
Connections:
- removed net N$20: ARD-SERVICE.TX, U$1.VCC1
- removed net N$6: PJ-320D.EARTH, V-IO.3
- new net 8V: 8V.P, MOLEX_0446200001.7, MOLEX_0446200001.8
- new net AUDIO: AUD.1, MOLEX_0446200001.5, PJ-320D.RING1, PJ-320D.TIP
- new net N$5: MINIMOSD.GND2, OSD-SERVICE.GND1
- new net V: ARD-SERVICE.TX, U$1.RX
- new net VMAIN: MOLEX_0446200001.3, PJ-320D.EARTH, V-IO.3
- net +5VFTDI: now also OSD-SERVICE.RX; no longer OSD-SERVICE.TX
- net DTR: now also OSD-SERVICE.1PPS; no longer OSD-SERVICE.GND1
- net GND: now also MOLEX_0446200001.2, MOLEX_0446200001.4; no longer OSD-SERVICE.1PPS, OSD-SERVICE.GND2
- net GPSTX: now also OSD-SERVICE.GND2; no longer OSD-SERVICE.VCC
- net N$12: now also U$1.A3; no longer U$1.A0
- net N$16: now also U$1.BLK; no longer U$1.DTR
- net N$18: now also U$1.GND0; no longer U$1.TX0-1
- net N$19: now also U$1.V; no longer U$1.RX1-1
- net N$21: now also U$1.TX; no longer U$1.GND4
- net N$3: now also MINIMOSD.GND1, OSD-SERVICE.VCC; no longer AUD.1, PJ-320D.RING1, PJ-320D.TIP
- net RX: now also OSD-SERVICE.TX; no longer OSD-SERVICE.RX
Other:
- note removed: "5:AUD"
- note removed: "6:NC"
- moved on the sheet: MOLEX_0446200001, SER
