File: eagle/PCB/PCB 2.brd (EAGLE design)
At the start: 45 x 75 mm, 7 parts

Commit message: More PCB work
Parts:
- removed IO2: (no value), con-lstb:MA07-1
- added J1: (no value), SparkFun-Connectors:1X04
- added J3: (no value), SparkFun-Connectors:1X03
- moved S1 2.84 mm to (14.0, 10.2)
Connections:
- removed net N$5: IO2.5, S2.3
- removed net N$8: IO2.6, S3.3
- removed net N$9: IO2.7, S4.3
- new net N$11: J3.2, S3.3
- new net N$12: J3.3, S2.3
- new net N$2: J3.1, S4.3
- net N$1: now also J1.2; no longer IO2.3
- net N$4: now also J1.1; no longer IO2.4
- net N$6: now also J1.4; no longer IO2.2
- net N$7: now also J1.3; no longer IO2.1
Changed lines of the file:
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@@
 <layer number="112" name="tSilk" color="7" fill="1" visible="no" active="yes"/>
 <layer number="113" name="ReferenceLS" color="7" fill="1" visible="no" active="no"/>
+<layer number="114" name="Badge_Outline" color="7" fill="1" visible="yes" active="yes"/>
+<layer number="115" name="ReferenceISLANDS" color="7" fill="1" visible="yes" active="yes"/>
 <layer number="116" name="Patch_BOT" color="9" fill="4" visible="no" active="yes"/>
 <layer number="118" name="Rect_Pads" color="7" fill="1" visible="no" active="no"/>
@@
 <vertex x="0" y="-0.123190625"/>
 </polygon>
-<text x="5.08" y="16.51" size="0.889" layer="25" rot="R270">SDA</text>
-<text x="5.08" y="19.05" size="0.889" layer="25" rot="R270">SCL</text>
-<text x="5.08" y="21.59" size="0.889" layer="25" rot="R270">G</text>
-<text x="5.08" y="24.13" size="0.889" layer="25" rot="R270">5V</text>
-<text x="5.08" y="26.67" size="0.889" layer="25" rot="R270">D2</text>
-<text x="5.08" y="29.21" size="0.889" layer="25" rot="R270">D3</text>
-<text x="5.08" y="31.75" size="0.889" layer="25" rot="R270">D4</text>
+<text x="5.08" y="21.59" size="0.889" layer="25" rot="R270">SDA</text>
+<text x="5.08" y="24.13" size="0.889" layer="25" rot="R270">SCL</text>
+<text x="5.08" y="17.78" size="0.889" layer="25" rot="R270">G</text>
+<text x="5.08" y="15.24" size="0.889" layer="25" rot="R270">5V</text>
+<text x="30.48" y="69.85" size="0.889" layer="25" rot="R270">D2</text>
+<text x="27.94" y="69.85" size="0.889" layer="25" rot="R270">D3</text>
+<text x="25.4" y="69.85" size="0.889" layer="25" rot="R270">D4</text>
 <text x="2.54" y="72.39" size="1.27" layer="26" rot="MR270">POCKET-GROUNDSTATION | PCB2 | REV1</text>
 <text x="38.1" y="3.81" size="0.889" layer="25" rot="R90">G</text>
@@
 </autorouter>
 <elements>
-<element name="IO2" library="con-lstb" library_urn="urn:adsk.eagle:library:162" package="MA07-1" package3d_urn="urn:adsk.eagle:package:8341/1" value="" x="2.54" y="24.13" smashed="yes" rot="R90">
-<attribute name="MF" value="" x="2.54" y="24.13" size="1.778" layer="27" rot="R90" display="off"/>
-<attribute name="MPN" value="" x="2.54" y="24.13" size="1.778" layer="27" rot="R90" display="off"/>
-<attribute name="OC_FARNELL" value="unknown" x="2.54" y="24.13" size="1.778" layer="27" rot="R90" display="off"/>
-<attribute name="OC_NEWARK" value="unknown" x="2.54" y="24.13" size="1.778" layer="27" rot="R90" display="off"/>
-<attribute name="VALUE" x="5.461" y="21.59" size="1.27" layer="27" ratio="10" rot="R90"/>
-</element>
 <element name="IO3" library="con-lstb" library_urn="urn:adsk.eagle:library:162" package="MA04-1" package3d_urn="urn:adsk.eagle:package:8337/1" value="" x="40.64" y="7.62" smashed="yes" rot="R90">
 <attribute name="MF" value="" x="40.64" y="7.62" size="1.778" layer="27" rot="R90" display="off"/>
@@
 <attribute name="VALUE" x="38.989" y="8.255" size="1.27" layer="27" ratio="10" rot="R90"/>
 </element>
-<element name="S1" library="switch" library_urn="urn:adsk.eagle:library:380" package="TL3XPO" package3d_urn="urn:adsk.eagle:package:27745/1" value="TL32PO" x="11.43" y="8.89" rot="R180"/>
+<element name="S1" library="switch" library_urn="urn:adsk.eagle:library:380" package="TL3XPO" package3d_urn="urn:adsk.eagle:package:27745/1" value="TL32PO" x="13.97" y="10.16" rot="R180"/>
 <element name="U$1" library="diy-modules" package="DISPLAY-OLED-128X64-I2C" value="DISPLAY-OLED-128X64-I2C" x="22.86" y="53.34" rot="R270"/>
 <element name="S2" library="SparkFun-Switches" library_urn="urn:adsk.eagle:library:535" package="TACTILE_SWITCH_PTH_6.0MM" package3d_urn="urn:adsk.eagle:package:40163/1" value="MOMENTARY-SWITCH-SPST-PTH-6.0MM" x="33.02" y="22.86">
@@
 <attribute name="SF_SKU" value="COM-00097" x="12.7" y="22.86" size="1.778" layer="27" display="off"/>
 </element>
+<element name="J1" library="SparkFun-Connectors" library_urn="urn:adsk.eagle:library:513" package="1X04" package3d_urn="urn:adsk.eagle:package:38085/1" value="" x="2.54" y="15.24" rot="R90">
+<attribute name="PROD_ID" value="CONN-09696" x="2.54" y="15.24" size="1.778" layer="27" rot="R90" display="off"/>
+</element>
+<element name="J3" library="SparkFun-Connectors" library_urn="urn:adsk.eagle:library:513" package="1X03" package3d_urn="urn:adsk.eagle:package:38063/1" value="" x="25.4" y="72.39"/>
 </elements>
 <signals>
@@
 <contactref element="IO3" pad="4"/>
 <contactref element="S1" pad="1"/>
-<wire x1="13.97" y1="8.89" x2="40.64" y2="11.43" width="0" layer="19" extent="1-1"/>
+<wire x1="16.51" y1="10.16" x2="40.64" y2="11.43" width="0" layer="19" extent="1-1"/>
 </signal>
 <signal name="N$3">
 <contactref element="IO3" pad="3"/>
 <contactref element="S1" pad="2"/>
-<wire x1="11.43" y1="8.89" x2="40.64" y2="8.89" width="0" layer="19" extent="1-1"/>
+<wire x1="13.97" y1="10.16" x2="40.64" y2="8.89" width="0" layer="19" extent="1-1"/>
 </signal>
 <signal name="N$1">
-<contactref element="IO2" pad="3"/>
 <contactref element="U$1" pad="1"/>
 <contactref element="IO3" pad="1"/>
@@
 <contactref element="S4" pad="1"/>
 <contactref element="S3" pad="1"/>
+<contactref element="J1" pad="2"/>
 <wire x1="29.7688" y1="25.1206" x2="35.56" y2="57.15" width="0" layer="19" extent="1-1"/>
 <wire x1="19.6088" y1="25.1206" x2="29.7688" y2="25.1206" width="0" layer="19" extent="1-1"/>
 <wire x1="9.4488" y1="25.1206" x2="19.6088" y2="25.1206" width="0" layer="19" extent="1-1"/>
-<wire x1="2.54" y1="21.59" x2="9.4488" y2="25.1206" width="0" layer="19" extent="1-1"/>
+<wire x1="2.54" y1="17.78" x2="9.4488" y2="25.1206" width="0" layer="19" extent="1-1"/>
 <wire x1="40.64" y1="3.81" x2="29.7688" y2="25.1206" width="0" layer="19" extent="1-1"/>
 </signal>
 <signal name="N$4">
 <contactref element="U$1" pad="2"/>
-<contactref element="IO2" pad="4"/>
-<wire x1="2.54" y1="24.13" x2="35.56" y2="54.61" width="0" layer="19" extent="1-1"/>
+<contactref element="J1" pad="1"/>
+<wire x1="2.54" y1="15.24" x2="35.56" y2="54.61" width="0" layer="19" extent="1-1"/>
 </signal>
 <signal name="N$6">
 <contactref element="U$1" pad="3"/>
-<contactref element="IO2" pad="2"/>
-<wire x1="2.54" y1="19.05" x2="35.56" y2="52.07" width="0" layer="19" extent="1-1"/>
+<contactref element="J1" pad="4"/>
+<wire x1="2.54" y1="22.86" x2="35.56" y2="52.07" width="0" layer="19" extent="1-1"/>
 </signal>
 <signal name="N$7">
 <contactref element="U$1" pad="4"/>
-<contactref element="IO2" pad="1"/>
-<wire x1="2.54" y1="16.51" x2="35.56" y2="49.53" width="0" layer="19" extent="1-1"/>
-</signal>
-<signal name="N$5">
-<contactref element="IO2" pad="5"/>
-<contactref element="S2" pad="3"/>
-<wire x1="2.54" y1="26.67" x2="29.7688" y2="20.5994" width="0" layer="19" extent="1-1"/>
-</signal>
-<signal name="N$8">
-<contactref element="IO2" pad="6"/>
-<contactref element="S3" pad="3"/>
-<wire x1="2.54" y1="29.21" x2="19.6088" y2="20.5994" width="0" layer="19" extent="1-1"/>
-</signal>
-<signal name="N$9">
-<contactref element="IO2" pad="7"/>
-<contactref element="S4" pad="3"/>
-<wire x1="9.4488" y1="20.5994" x2="2.54" y2="31.75" width="0" layer="19" extent="1-1"/>
+<contactref element="J1" pad="3"/>
+<wire x1="2.54" y1="20.32" x2="35.56" y2="49.53" width="0" layer="19" extent="1-1"/>
 </signal>
 <signal name="N$10">
 <contactref element="IO3" pad="2"/>
 <contactref element="S1" pad="3"/>
-<wire x1="8.89" y1="8.89" x2="40.64" y2="6.35" width="0" layer="19" extent="1-1"/>
+<wire x1="11.43" y1="10.16" x2="40.64" y2="6.35" width="0" layer="19" extent="1-1"/>
+</signal>
+<signal name="N$2">
+<contactref element="S4" pad="3"/>
+<contactref element="J3" pad="1"/>
+<wire x1="9.4488" y1="20.5994" x2="25.4" y2="72.39" width="0" layer="19" extent="1-1"/>
+</signal>
+<signal name="N$11">
+<contactref element="S3" pad="3"/>
+<contactref element="J3" pad="2"/>
+<wire x1="19.6088" y1="20.5994" x2="27.94" y2="72.39" width="0" layer="19" extent="1-1"/>
+</signal>
+<signal name="N$12">
+<contactref element="S2" pad="3"/>
+<contactref element="J3" pad="3"/>
+<wire x1="29.7688" y1="20.5994" x2="30.48" y2="72.39" width="0" layer="19" extent="1-1"/>
 </signal>
 </signals>
