File: eagle/PCB/PCB 2.brd (EAGLE design)
At the start: 45 x 75 mm, 8 parts

Commit message: PCB Work
Parts:
- removed U$1: DISPLAY-OLED-128X64-I2C, diy-modules:DISPLAY-OLED-128X64-I2C
- added OLED: DISPLAY-OLED-128X64-I2C, diy-modules:DISPLAY-OLED-128X64-I2C
- added U$2, U$3, U$4, U$5: (no value), holes:3,0
- moved IO3 7.62 mm to (40.6, 15.2)
- moved S2 1.27 mm to (31.8, 22.9)
- moved S4 1.27 mm to (14.0, 22.9)
Connections:
- net N$1: now also OLED.1; no longer U$1.1
- net N$4: now also OLED.2; no longer U$1.2
- net N$6: now also OLED.4; no longer U$1.4
- net N$7: now also OLED.3; no longer U$1.3
Changed lines of the file:
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@@
 <text x="25.4" y="69.85" size="0.889" layer="25" rot="R270">D4</text>
 <text x="2.54" y="72.39" size="1.27" layer="26" rot="MR270">POCKET-GROUNDSTATION | PCB2 | REV1</text>
-<text x="38.1" y="3.81" size="0.889" layer="25" rot="R90">G</text>
-<text x="38.1" y="6.35" size="0.889" layer="25" rot="R180">Vdvr</text>
-<text x="38.1" y="8.89" size="0.889" layer="25" rot="R180">Vmain</text>
-<text x="38.1" y="11.43" size="0.889" layer="25" rot="R180">Vosd</text>
+<text x="38.1" y="11.43" size="0.889" layer="25" rot="R180">G</text>
+<text x="38.1" y="13.97" size="0.889" layer="25" rot="R180">Vdvr</text>
+<text x="38.1" y="16.51" size="0.889" layer="25" rot="R180">Vmain</text>
+<text x="38.1" y="19.05" size="0.889" layer="25" rot="R180">Vosd</text>
 </plain>
 <attributes>
@@
 </autorouter>
 <elements>
-<element name="IO3" library="con-lstb" library_urn="urn:adsk.eagle:library:162" package="MA04-1" package3d_urn="urn:adsk.eagle:package:8337/1" value="" x="40.64" y="7.62" smashed="yes" rot="R90">
-<attribute name="MF" value="" x="40.64" y="7.62" size="1.778" layer="27" rot="R90" display="off"/>
-<attribute name="MPN" value="" x="40.64" y="7.62" size="1.778" layer="27" rot="R90" display="off"/>
-<attribute name="OC_FARNELL" value="unknown" x="40.64" y="7.62" size="1.778" layer="27" rot="R90" display="off"/>
-<attribute name="OC_NEWARK" value="unknown" x="40.64" y="7.62" size="1.778" layer="27" rot="R90" display="off"/>
-<attribute name="VALUE" x="38.989" y="8.255" size="1.27" layer="27" ratio="10" rot="R90"/>
+<element name="IO3" library="con-lstb" library_urn="urn:adsk.eagle:library:162" package="MA04-1" package3d_urn="urn:adsk.eagle:package:8337/1" value="" x="40.64" y="15.24" smashed="yes" rot="R90">
+<attribute name="MF" value="" x="40.64" y="15.24" size="1.778" layer="27" rot="R90" display="off"/>
+<attribute name="MPN" value="" x="40.64" y="15.24" size="1.778" layer="27" rot="R90" display="off"/>
+<attribute name="OC_FARNELL" value="unknown" x="40.64" y="15.24" size="1.778" layer="27" rot="R90" display="off"/>
+<attribute name="OC_NEWARK" value="unknown" x="40.64" y="15.24" size="1.778" layer="27" rot="R90" display="off"/>
+<attribute name="VALUE" x="38.989" y="15.875" size="1.27" layer="27" ratio="10" rot="R90"/>
 </element>
 <element name="S1" library="switch" library_urn="urn:adsk.eagle:library:380" package="TL3XPO" package3d_urn="urn:adsk.eagle:package:27745/1" value="TL32PO" x="13.97" y="10.16" rot="R180"/>
-<element name="U$1" library="diy-modules" package="DISPLAY-OLED-128X64-I2C" value="DISPLAY-OLED-128X64-I2C" x="22.86" y="53.34" rot="R270"/>
-<element name="S2" library="SparkFun-Switches" library_urn="urn:adsk.eagle:library:535" package="TACTILE_SWITCH_PTH_6.0MM" package3d_urn="urn:adsk.eagle:package:40163/1" value="MOMENTARY-SWITCH-SPST-PTH-6.0MM" x="33.02" y="22.86">
-<attribute name="PROD_ID" value=" SWCH-08441" x="33.02" y="22.86" size="1.778" layer="27" display="off"/>
-<attribute name="SF_SKU" value="COM-00097" x="33.02" y="22.86" size="1.778" layer="27" display="off"/>
+<element name="OLED" library="diy-modules" package="DISPLAY-OLED-128X64-I2C" value="DISPLAY-OLED-128X64-I2C" x="22.86" y="50.8" rot="R270"/>
+<element name="S2" library="SparkFun-Switches" library_urn="urn:adsk.eagle:library:535" package="TACTILE_SWITCH_PTH_6.0MM" package3d_urn="urn:adsk.eagle:package:40163/1" value="MOMENTARY-SWITCH-SPST-PTH-6.0MM" x="31.75" y="22.86">
+<attribute name="PROD_ID" value=" SWCH-08441" x="31.75" y="22.86" size="1.778" layer="27" display="off"/>
+<attribute name="SF_SKU" value="COM-00097" x="31.75" y="22.86" size="1.778" layer="27" display="off"/>
 </element>
 <element name="S3" library="SparkFun-Switches" library_urn="urn:adsk.eagle:library:535" package="TACTILE_SWITCH_PTH_6.0MM" package3d_urn="urn:adsk.eagle:package:40163/1" value="MOMENTARY-SWITCH-SPST-PTH-6.0MM" x="22.86" y="22.86">
@@
 <attribute name="SF_SKU" value="COM-00097" x="22.86" y="22.86" size="1.778" layer="27" display="off"/>
 </element>
-<element name="S4" library="SparkFun-Switches" library_urn="urn:adsk.eagle:library:535" package="TACTILE_SWITCH_PTH_6.0MM" package3d_urn="urn:adsk.eagle:package:40163/1" value="MOMENTARY-SWITCH-SPST-PTH-6.0MM" x="12.7" y="22.86">
-<attribute name="PROD_ID" value=" SWCH-08441" x="12.7" y="22.86" size="1.778" layer="27" display="off"/>
-<attribute name="SF_SKU" value="COM-00097" x="12.7" y="22.86" size="1.778" layer="27" display="off"/>
+<element name="S4" library="SparkFun-Switches" library_urn="urn:adsk.eagle:library:535" package="TACTILE_SWITCH_PTH_6.0MM" package3d_urn="urn:adsk.eagle:package:40163/1" value="MOMENTARY-SWITCH-SPST-PTH-6.0MM" x="13.97" y="22.86">
+<attribute name="PROD_ID" value=" SWCH-08441" x="13.97" y="22.86" size="1.778" layer="27" display="off"/>
+<attribute name="SF_SKU" value="COM-00097" x="13.97" y="22.86" size="1.778" layer="27" display="off"/>
 </element>
 <element name="J1" library="SparkFun-Connectors" library_urn="urn:adsk.eagle:library:513" package="1X04" package3d_urn="urn:adsk.eagle:package:38085/1" value="" x="2.54" y="15.24" rot="R90">
@@
 </element>
 <element name="J3" library="SparkFun-Connectors" library_urn="urn:adsk.eagle:library:513" package="1X03" package3d_urn="urn:adsk.eagle:package:38063/1" value="" x="25.4" y="72.39"/>
+<element name="U$2" library="holes" library_urn="urn:adsk.eagle:library:237" package="3,0" package3d_urn="urn:adsk.eagle:package:14277/1" value="" x="5.08" y="69.85"/>
+<element name="U$3" library="holes" library_urn="urn:adsk.eagle:library:237" package="3,0" package3d_urn="urn:adsk.eagle:package:14277/1" value="" x="40.64" y="69.85"/>
+<element name="U$4" library="holes" library_urn="urn:adsk.eagle:library:237" package="3,0" package3d_urn="urn:adsk.eagle:package:14277/1" value="" x="5.08" y="5.08"/>
+<element name="U$5" library="holes" library_urn="urn:adsk.eagle:library:237" package="3,0" package3d_urn="urn:adsk.eagle:package:14277/1" value="" x="40.64" y="5.08"/>
 </elements>
 <signals>
@@
 <contactref element="IO3" pad="4"/>
 <contactref element="S1" pad="1"/>
-<wire x1="16.51" y1="10.16" x2="40.64" y2="11.43" width="0" layer="19" extent="1-1"/>
+<wire x1="16.51" y1="10.16" x2="40.64" y2="19.05" width="0" layer="19" extent="1-1"/>
 </signal>
 <signal name="N$3" class="2">
 <contactref element="IO3" pad="3"/>
 <contactref element="S1" pad="2"/>
-<wire x1="13.97" y1="10.16" x2="40.64" y2="8.89" width="0" layer="19" extent="1-1"/>
+<wire x1="13.97" y1="10.16" x2="40.64" y2="16.51" width="0" layer="19" extent="1-1"/>
 </signal>
 <signal name="N$1">
-<contactref element="U$1" pad="1"/>
+<contactref element="OLED" pad="1"/>
 <contactref element="IO3" pad="1"/>
 <contactref element="S2" pad="1"/>
@@
 <contactref element="S3" pad="1"/>
 <contactref element="J1" pad="2"/>
-<wire x1="29.7688" y1="25.1206" x2="35.56" y2="57.15" width="0" layer="19" extent="1-1"/>
-<wire x1="19.6088" y1="25.1206" x2="29.7688" y2="25.1206" width="0" layer="19" extent="1-1"/>
-<wire x1="9.4488" y1="25.1206" x2="19.6088" y2="25.1206" width="0" layer="19" extent="1-1"/>
-<wire x1="2.54" y1="17.78" x2="9.4488" y2="25.1206" width="0" layer="19" extent="1-1"/>
-<wire x1="40.64" y1="3.81" x2="29.7688" y2="25.1206" width="0" layer="19" extent="1-1"/>
+<wire x1="28.4988" y1="25.1206" x2="35.56" y2="54.61" width="0" layer="19" extent="1-1"/>
+<wire x1="19.6088" y1="25.1206" x2="28.4988" y2="25.1206" width="0" layer="19" extent="1-1"/>
+<wire x1="10.7188" y1="25.1206" x2="19.6088" y2="25.1206" width="0" layer="19" extent="1-1"/>
+<wire x1="2.54" y1="17.78" x2="10.7188" y2="25.1206" width="0" layer="19" extent="1-1"/>
+<wire x1="40.64" y1="11.43" x2="28.4988" y2="25.1206" width="0" layer="19" extent="1-1"/>
 </signal>
 <signal name="N$4">
-<contactref element="U$1" pad="2"/>
+<contactref element="OLED" pad="2"/>
 <contactref element="J1" pad="1"/>
-<wire x1="2.54" y1="15.24" x2="35.56" y2="54.61" width="0" layer="19" extent="1-1"/>
+<wire x1="2.54" y1="15.24" x2="35.56" y2="52.07" width="0" layer="19" extent="1-1"/>
 </signal>
 <signal name="N$6" class="1">
 <contactref element="J1" pad="4"/>
-<contactref element="U$1" pad="4"/>
-<wire x1="2.54" y1="22.86" x2="35.56" y2="49.53" width="0" layer="19" extent="1-1"/>
+<contactref element="OLED" pad="4"/>
+<wire x1="2.54" y1="22.86" x2="35.56" y2="46.99" width="0" layer="19" extent="1-1"/>
 </signal>
 <signal name="N$7" class="1">
 <contactref element="J1" pad="3"/>
-<contactref element="U$1" pad="3"/>
-<wire x1="2.54" y1="20.32" x2="35.56" y2="52.07" width="0" layer="19" extent="1-1"/>
+<contactref element="OLED" pad="3"/>
+<wire x1="2.54" y1="20.32" x2="35.56" y2="49.53" width="0" layer="19" extent="1-1"/>
 </signal>
 <signal name="N$10" class="2">
 <contactref element="IO3" pad="2"/>
 <contactref element="S1" pad="3"/>
-<wire x1="11.43" y1="10.16" x2="40.64" y2="6.35" width="0" layer="19" extent="1-1"/>
+<wire x1="11.43" y1="10.16" x2="40.64" y2="13.97" width="0" layer="19" extent="1-1"/>
 </signal>
 <signal name="N$2" class="1">
 <contactref element="S4" pad="3"/>
 <contactref element="J3" pad="1"/>
-<wire x1="9.4488" y1="20.5994" x2="25.4" y2="72.39" width="0" layer="19" extent="1-1"/>
+<wire x1="10.7188" y1="20.5994" x2="25.4" y2="72.39" width="0" layer="19" extent="1-1"/>
 </signal>
 <signal name="N$11" class="1">
@@
 <contactref element="S2" pad="3"/>
 <contactref element="J3" pad="3"/>
-<wire x1="29.7688" y1="20.5994" x2="30.48" y2="72.39" width="0" layer="19" extent="1-1"/>
+<wire x1="28.4988" y1="20.5994" x2="30.48" y2="72.39" width="0" layer="19" extent="1-1"/>
 </signal>
 </signals>

Commit message: PCB updates
Parts:
- removed J3: (no value), SparkFun-Connectors:1X03
- added BT-IO: (no value), SparkFun-Connectors:1X04
- added D1: (no value), SparkFun-LED:LED_3MM
- added R3-220: 220, resistor:R1206
- moved S1 53.4 mm to (16.5, 63.5)
- moved OLED 12.8 mm to (24.1, 38.1)
- moved S2 10.2 mm to (31.8, 12.7)
- moved S3 10.2 mm to (22.9, 12.7)
- moved S4 10.2 mm to (14.0, 12.7)
- moved U$4 1.49 mm to (4.88, 3.61)
- moved U$2 1.27 mm to (5.08, 71.1)
- moved U$3 1.27 mm to (40.6, 71.1)
- moved U$5 1.27 mm to (40.6, 3.81)
- renumbered J1 to OLED-IO
Connections:
- new net GND: D1.K, IO3.1, OLED-IO.2, OLED.1, S2.1, S3.1, S4.1
- new net N$5: BT-IO.4, R3-220.1
- net N$1: now also D1.A, R3-220.2; no longer IO3.1, OLED-IO.2, OLED.1, S2.1, S3.1, S4.1
- net N$11: now also BT-IO.2; no longer J3.2
- net N$12: now also BT-IO.3; no longer J3.3
- net N$2: now also BT-IO.1; no longer J3.1
Other:
- board text added: "D13 (LED)"

Commit message: small PCB updates
Parts:
- moved U$2 0.76 mm to (4.32, 71.1)
- moved U$4 0.59 mm to (4.32, 3.81)
Changed lines of the file:
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@@
 <attribute name="PROD_ID" value="CONN-09696" x="24.13" y="72.39" size="1.778" layer="27" display="off"/>
 </element>
-<element name="U$2" library="holes" library_urn="urn:adsk.eagle:library:237" package="3,0" package3d_urn="urn:adsk.eagle:package:14277/1" value="" x="5.08" y="71.12"/>
+<element name="U$2" library="holes" library_urn="urn:adsk.eagle:library:237" package="3,0" package3d_urn="urn:adsk.eagle:package:14277/1" value="" x="4.318" y="71.12"/>
 <element name="U$3" library="holes" library_urn="urn:adsk.eagle:library:237" package="3,0" package3d_urn="urn:adsk.eagle:package:14277/1" value="" x="40.64" y="71.12"/>
-<element name="U$4" library="holes" library_urn="urn:adsk.eagle:library:237" package="3,0" package3d_urn="urn:adsk.eagle:package:14277/1" value="" x="4.8768" y="3.6068"/>
+<element name="U$4" library="holes" library_urn="urn:adsk.eagle:library:237" package="3,0" package3d_urn="urn:adsk.eagle:package:14277/1" value="" x="4.318" y="3.81"/>
 <element name="U$5" library="holes" library_urn="urn:adsk.eagle:library:237" package="3,0" package3d_urn="urn:adsk.eagle:package:14277/1" value="" x="40.64" y="3.81"/>
 <element name="D1" library="SparkFun-LED" library_urn="urn:adsk.eagle:library:529" package="LED_3MM" package3d_urn="urn:adsk.eagle:package:39361/1" value="" x="31.75" y="63.5">
