File: eagle/PCB/PCB 2.sch (EAGLE design)
At the start: 7 parts

Commit message: More PCB work
Parts:
- removed IO2: (no value), con-lstb:MA07-1
- added J1: (no value), SparkFun-Connectors:CONN_04
- added J3: (no value), SparkFun-Connectors:CONN_03
Connections:
- removed net N$5: IO2.5, S2.2
- removed net N$8: IO2.6, S3.2
- removed net N$9: IO2.7, S4.2
- new net N$11: J3.2, S3.2
- new net N$12: J3.3, S2.2
- new net N$2: J3.1, S4.2
- net N$1: now also J1.2; no longer IO2.3
- net N$4: now also J1.1; no longer IO2.4
- net N$6: now also J1.4; no longer IO2.2
- net N$7: now also J1.3; no longer IO2.1
Other:
- moved on the sheet: S2, S3
Changed lines of the file:
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@@
 <layer number="112" name="tSilk" color="7" fill="1" visible="no" active="yes"/>
 <layer number="113" name="ReferenceLS" color="7" fill="1" visible="no" active="no"/>
+<layer number="114" name="Badge_Outline" color="7" fill="1" visible="yes" active="yes"/>
+<layer number="115" name="ReferenceISLANDS" color="7" fill="1" visible="yes" active="yes"/>
 <layer number="116" name="Patch_BOT" color="9" fill="4" visible="yes" active="yes"/>
 <layer number="118" name="Rect_Pads" color="7" fill="1" visible="no" active="no"/>
@@
 </classes>
 <parts>
-<part name="IO2" library="con-lstb" library_urn="urn:adsk.eagle:library:162" deviceset="MA07-1" device="" package3d_urn="urn:adsk.eagle:package:8341/1"/>
 <part name="IO3" library="con-lstb" library_urn="urn:adsk.eagle:library:162" deviceset="MA04-1" device="" package3d_urn="urn:adsk.eagle:package:8337/1"/>
 <part name="S1" library="switch" library_urn="urn:adsk.eagle:library:380" deviceset="TL32PO" device="" package3d_urn="urn:adsk.eagle:package:27745/1"/>
@@
 <part name="S3" library="SparkFun-Switches" library_urn="urn:adsk.eagle:library:535" deviceset="MOMENTARY-SWITCH-SPST" device="-PTH-6.0MM" package3d_urn="urn:adsk.eagle:package:40163/1"/>
 <part name="S4" library="SparkFun-Switches" library_urn="urn:adsk.eagle:library:535" deviceset="MOMENTARY-SWITCH-SPST" device="-PTH-6.0MM" package3d_urn="urn:adsk.eagle:package:40163/1"/>
+<part name="J1" library="SparkFun-Connectors" library_urn="urn:adsk.eagle:library:513" deviceset="CONN_04" device="" package3d_urn="urn:adsk.eagle:package:38085/1"/>
+<part name="J3" library="SparkFun-Connectors" library_urn="urn:adsk.eagle:library:513" deviceset="CONN_03" device="" package3d_urn="urn:adsk.eagle:package:38063/1"/>
 </parts>
 <sheets>
@@
 <text x="104.14" y="142.24" size="1.778" layer="91" rot="R180">VO DVR</text>
 <text x="104.14" y="139.7" size="1.778" layer="91" rot="R180">GND</text>
-<text x="93.98" y="198.12" size="1.778" layer="91" rot="R90">SDA (A4) </text>
-<text x="96.52" y="198.12" size="1.778" layer="91" rot="R90">SCL (A6)</text>
-<text x="99.06" y="198.12" size="1.778" layer="91" rot="R90">GND</text>
-<text x="101.6" y="198.12" size="1.778" layer="91" rot="R90">5V</text>
-<text x="104.14" y="198.12" size="1.778" layer="91" rot="R90">D2</text>
-<text x="106.68" y="198.12" size="1.778" layer="91" rot="R90">D3</text>
-<text x="109.22" y="198.12" size="1.778" layer="91" rot="R90">D4</text>
+<text x="101.6" y="198.12" size="1.778" layer="91" rot="R90">SDA (A4) </text>
+<text x="99.06" y="198.12" size="1.778" layer="91" rot="R90">SCL (A6)</text>
+<text x="96.52" y="198.12" size="1.778" layer="91" rot="R90">GND</text>
+<text x="93.98" y="198.12" size="1.778" layer="91" rot="R90">5V</text>
+<text x="60.96" y="218.44" size="1.778" layer="91" rot="R90">D2</text>
+<text x="63.5" y="218.44" size="1.778" layer="91" rot="R90">D3</text>
+<text x="66.04" y="218.44" size="1.778" layer="91" rot="R90">D4</text>
 </plain>
 <instances>
-<instance part="IO2" gate="1" x="101.6" y="195.58" smashed="yes" rot="R270">
-<attribute name="VALUE" x="88.9" y="196.85" size="1.778" layer="96" rot="R270"/>
-</instance>
 <instance part="IO3" gate="1" x="106.68" y="144.78" smashed="yes">
 <attribute name="VALUE" x="105.41" y="132.08" size="1.778" layer="96"/>
@@
 <instance part="S1" gate="BEF1" x="144.78" y="132.08" rot="R180"/>
 <instance part="U$1" gate="G$1" x="160.02" y="175.26"/>
-<instance part="S2" gate="G$1" x="66.04" y="170.18" rot="R90"/>
-<instance part="S3" gate="G$1" x="60.96" y="172.72" rot="R90"/>
+<instance part="S2" gate="G$1" x="63.5" y="170.18" rot="R90"/>
+<instance part="S3" gate="G$1" x="58.42" y="172.72" rot="R90"/>
 <instance part="S4" gate="G$1" x="53.34" y="175.26" rot="R90"/>
+<instance part="J1" gate="G$1" x="96.52" y="190.5" rot="R270"/>
+<instance part="J3" gate="J$1" x="60.96" y="213.36" rot="R270"/>
 </instances>
 <busses>
@@
 <net name="N$1" class="0">
 <segment>
-<pinref part="IO2" gate="1" pin="3"/>
-<wire x1="99.06" y1="187.96" x2="99.06" y2="172.72" width="0.1524" layer="91"/>
 <wire x1="99.06" y1="172.72" x2="99.06" y2="170.18" width="0.1524" layer="91"/>
 <wire x1="99.06" y1="170.18" x2="116.84" y2="170.18" width="0.1524" layer="91"/>
@@
 <pinref part="U$1" gate="G$1" pin="GND"/>
 <wire x1="154.94" y1="198.12" x2="154.94" y2="195.58" width="0.1524" layer="91"/>
-<wire x1="99.06" y1="172.72" x2="71.12" y2="172.72" width="0.1524" layer="91"/>
-<junction x="99.06" y="172.72"/>
 <pinref part="IO3" gate="1" pin="1"/>
+<wire x1="99.06" y1="172.72" x2="96.52" y2="172.72" width="0.1524" layer="91"/>
+<wire x1="96.52" y1="172.72" x2="71.12" y2="172.72" width="0.1524" layer="91"/>
 <wire x1="116.84" y1="139.7" x2="114.3" y2="139.7" width="0.1524" layer="91"/>
 <wire x1="116.84" y1="139.7" x2="116.84" y2="170.18" width="0.1524" layer="91"/>
@@
 <wire x1="71.12" y1="172.72" x2="71.12" y2="165.1" width="0.1524" layer="91"/>
 <pinref part="S2" gate="G$1" pin="1"/>
-<wire x1="71.12" y1="165.1" x2="66.04" y2="165.1" width="0.1524" layer="91"/>
-<wire x1="66.04" y1="165.1" x2="60.96" y2="165.1" width="0.1524" layer="91"/>
-<junction x="66.04" y="165.1"/>
+<wire x1="71.12" y1="165.1" x2="63.5" y2="165.1" width="0.1524" layer="91"/>
+<wire x1="63.5" y1="165.1" x2="58.42" y2="165.1" width="0.1524" layer="91"/>
+<junction x="63.5" y="165.1"/>
 <pinref part="S4" gate="G$1" pin="1"/>
-<wire x1="60.96" y1="165.1" x2="53.34" y2="165.1" width="0.1524" layer="91"/>
+<wire x1="58.42" y1="165.1" x2="53.34" y2="165.1" width="0.1524" layer="91"/>
 <wire x1="53.34" y1="165.1" x2="53.34" y2="170.18" width="0.1524" layer="91"/>
 <pinref part="S3" gate="G$1" pin="1"/>
-<wire x1="60.96" y1="165.1" x2="60.96" y2="167.64" width="0.1524" layer="91"/>
-<junction x="60.96" y="165.1"/>
+<wire x1="58.42" y1="165.1" x2="58.42" y2="167.64" width="0.1524" layer="91"/>
+<junction x="58.42" y="165.1"/>
+<pinref part="J1" gate="G$1" pin="2"/>
+<wire x1="96.52" y1="185.42" x2="96.52" y2="172.72" width="0.1524" layer="91"/>
+<junction x="96.52" y="172.72"/>
 </segment>
 </net>
@@
 <wire x1="157.48" y1="200.66" x2="121.92" y2="200.66" width="0.1524" layer="91"/>
 <wire x1="121.92" y1="200.66" x2="121.92" y2="172.72" width="0.1524" layer="91"/>
-<pinref part="IO2" gate="1" pin="4"/>
-<wire x1="101.6" y1="187.96" x2="101.6" y2="172.72" width="0.1524" layer="91"/>
 <wire x1="101.6" y1="172.72" x2="121.92" y2="172.72" width="0.1524" layer="91"/>
+<wire x1="101.6" y1="172.72" x2="101.6" y2="175.26" width="0.1524" layer="91"/>
+<wire x1="101.6" y1="175.26" x2="93.98" y2="175.26" width="0.1524" layer="91"/>
+<pinref part="J1" gate="G$1" pin="1"/>
+<wire x1="93.98" y1="185.42" x2="93.98" y2="175.26" width="0.1524" layer="91"/>
 </segment>
 </net>
@@
 <wire x1="208.28" y1="198.12" x2="208.28" y2="172.72" width="0.1524" layer="91"/>
 <wire x1="208.28" y1="172.72" x2="187.96" y2="152.4" width="0.1524" layer="91"/>
-<wire x1="187.96" y1="152.4" x2="96.52" y2="152.4" width="0.1524" layer="91"/>
-<pinref part="IO2" gate="1" pin="2"/>
-<wire x1="96.52" y1="152.4" x2="96.52" y2="187.96" width="0.1524" layer="91"/>
+<wire x1="187.96" y1="152.4" x2="81.28" y2="152.4" width="0.1524" layer="91"/>
+<pinref part="J1" gate="G$1" pin="4"/>
+<wire x1="101.6" y1="185.42" x2="101.6" y2="182.88" width="0.1524" layer="91"/>
+<wire x1="101.6" y1="182.88" x2="81.28" y2="182.88" width="0.1524" layer="91"/>
+<wire x1="81.28" y1="182.88" x2="81.28" y2="152.4" width="0.1524" layer="91"/>
 </segment>
 </net>
@@
 <wire x1="205.74" y1="175.26" x2="205.74" y2="195.58" width="0.1524" layer="91"/>
 <wire x1="205.74" y1="175.26" x2="185.42" y2="154.94" width="0.1524" layer="91"/>
-<wire x1="185.42" y1="154.94" x2="93.98" y2="154.94" width="0.1524" layer="91"/>
-<pinref part="IO2" gate="1" pin="1"/>
-<wire x1="93.98" y1="154.94" x2="93.98" y2="187.96" width="0.1524" layer="91"/>
-</segment>
-</net>
-<net name="N$5" class="0">
-<segment>
-<pinref part="IO2" gate="1" pin="5"/>
-<wire x1="104.14" y1="187.96" x2="104.14" y2="175.26" width="0.1524" layer="91"/>
-<wire x1="104.14" y1="175.26" x2="66.04" y2="175.26" width="0.1524" layer="91"/>
-<pinref part="S2" gate="G$1" pin="2"/>
-</segment>
-</net>
-<net name="N$8" class="0">
-<segment>
-<pinref part="IO2" gate="1" pin="6"/>
-<wire x1="106.68" y1="187.96" x2="106.68" y2="177.8" width="0.1524" layer="91"/>
-<wire x1="106.68" y1="177.8" x2="60.96" y2="177.8" width="0.1524" layer="91"/>
-<pinref part="S3" gate="G$1" pin="2"/>
-</segment>
-</net>
-<net name="N$9" class="0">
-<segment>
-<pinref part="IO2" gate="1" pin="7"/>
-<wire x1="109.22" y1="187.96" x2="109.22" y2="180.34" width="0.1524" layer="91"/>
-<wire x1="109.22" y1="180.34" x2="53.34" y2="180.34" width="0.1524" layer="91"/>
-<pinref part="S4" gate="G$1" pin="2"/>
+<wire x1="185.42" y1="154.94" x2="86.36" y2="154.94" width="0.1524" layer="91"/>
+<pinref part="J1" gate="G$1" pin="3"/>
+<wire x1="99.06" y1="185.42" x2="99.06" y2="180.34" width="0.1524" layer="91"/>
+<wire x1="99.06" y1="180.34" x2="86.36" y2="180.34" width="0.1524" layer="91"/>
+<wire x1="86.36" y1="180.34" x2="86.36" y2="154.94" width="0.1524" layer="91"/>
 </segment>
 </net>
@@
 </segment>
 </net>
+<net name="N$2" class="0">
+<segment>
+<pinref part="S4" gate="G$1" pin="2"/>
+<pinref part="J3" gate="J$1" pin="1"/>
+<wire x1="53.34" y1="180.34" x2="58.42" y2="180.34" width="0.1524" layer="91"/>
+<wire x1="58.42" y1="180.34" x2="58.42" y2="205.74" width="0.1524" layer="91"/>
+</segment>
+</net>
+<net name="N$11" class="0">
+<segment>
+<pinref part="S3" gate="G$1" pin="2"/>
+<pinref part="J3" gate="J$1" pin="2"/>
+<wire x1="58.42" y1="177.8" x2="60.96" y2="177.8" width="0.1524" layer="91"/>
+<wire x1="60.96" y1="177.8" x2="60.96" y2="205.74" width="0.1524" layer="91"/>
+</segment>
+</net>
+<net name="N$12" class="0">
+<segment>
+<pinref part="S2" gate="G$1" pin="2"/>
+<pinref part="J3" gate="J$1" pin="3"/>
+<wire x1="63.5" y1="175.26" x2="63.5" y2="205.74" width="0.1524" layer="91"/>
+</segment>
+</net>
