File: eagle/PCB/PCB 2.sch (EAGLE design)
At the start: 8 parts

Commit message: PCB Work
Parts:
- renumbered U$1 to OLED
Changed lines of the file:
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@@
 <part name="IO3" library="con-lstb" library_urn="urn:adsk.eagle:library:162" deviceset="MA04-1" device="" package3d_urn="urn:adsk.eagle:package:8337/1"/>
 <part name="S1" library="switch" library_urn="urn:adsk.eagle:library:380" deviceset="TL32PO" device="" package3d_urn="urn:adsk.eagle:package:27745/1"/>
-<part name="U$1" library="diy-modules" deviceset="DISPLAY-OLED-128X64-I2C" device=""/>
+<part name="OLED" library="diy-modules" deviceset="DISPLAY-OLED-128X64-I2C" device=""/>
 <part name="S2" library="SparkFun-Switches" library_urn="urn:adsk.eagle:library:535" deviceset="MOMENTARY-SWITCH-SPST" device="-PTH-6.0MM" package3d_urn="urn:adsk.eagle:package:40163/1"/>
 <part name="S3" library="SparkFun-Switches" library_urn="urn:adsk.eagle:library:535" deviceset="MOMENTARY-SWITCH-SPST" device="-PTH-6.0MM" package3d_urn="urn:adsk.eagle:package:40163/1"/>
@@
 </instance>
 <instance part="S1" gate="BEF1" x="144.78" y="132.08" rot="R180"/>
-<instance part="U$1" gate="G$1" x="160.02" y="175.26"/>
+<instance part="OLED" gate="G$1" x="160.02" y="175.26"/>
 <instance part="S2" gate="G$1" x="63.5" y="170.18" rot="R90"/>
 <instance part="S3" gate="G$1" x="58.42" y="172.72" rot="R90"/>
@@
 <wire x1="124.46" y1="170.18" x2="124.46" y2="198.12" width="0.1524" layer="91"/>
 <wire x1="124.46" y1="198.12" x2="154.94" y2="198.12" width="0.1524" layer="91"/>
-<pinref part="U$1" gate="G$1" pin="GND"/>
+<pinref part="OLED" gate="G$1" pin="GND"/>
 <wire x1="154.94" y1="198.12" x2="154.94" y2="195.58" width="0.1524" layer="91"/>
 <pinref part="IO3" gate="1" pin="1"/>
@@
 <net name="N$4" class="0">
 <segment>
-<pinref part="U$1" gate="G$1" pin="VCC"/>
+<pinref part="OLED" gate="G$1" pin="VCC"/>
 <wire x1="157.48" y1="195.58" x2="157.48" y2="200.66" width="0.1524" layer="91"/>
 <wire x1="157.48" y1="200.66" x2="121.92" y2="200.66" width="0.1524" layer="91"/>
@@
 <wire x1="101.6" y1="182.88" x2="81.28" y2="182.88" width="0.1524" layer="91"/>
 <wire x1="81.28" y1="182.88" x2="81.28" y2="152.4" width="0.1524" layer="91"/>
-<pinref part="U$1" gate="G$1" pin="SDA"/>
+<pinref part="OLED" gate="G$1" pin="SDA"/>
 <wire x1="208.28" y1="208.28" x2="162.56" y2="208.28" width="0.1524" layer="91"/>
 <wire x1="162.56" y1="208.28" x2="162.56" y2="195.58" width="0.1524" layer="91"/>
@@
 <wire x1="86.36" y1="180.34" x2="86.36" y2="154.94" width="0.1524" layer="91"/>
 <wire x1="205.74" y1="198.12" x2="160.02" y2="198.12" width="0.1524" layer="91"/>
-<pinref part="U$1" gate="G$1" pin="SCL"/>
+<pinref part="OLED" gate="G$1" pin="SCL"/>
 <wire x1="160.02" y1="198.12" x2="160.02" y2="195.58" width="0.1524" layer="91"/>
 </segment>

Commit message: PCB updates
Parts:
- removed J3: (no value), SparkFun-Connectors:CONN_03
- added BT-IO: (no value), SparkFun-Connectors:CONN_04
- added D1: (no value), SparkFun-LED:LED3MM
- added R3-220: 220, resistor:R-EU_R1206
- renumbered J1 to OLED-IO
Connections:
- new net GND: D1.C, IO3.1, OLED-IO.2, OLED.GND, S2.1, S3.1, S4.1
- new net N$5: BT-IO.4, R3-220.1
- net N$1: now also D1.A, R3-220.2; no longer IO3.1, OLED-IO.2, OLED.GND, S2.1, S3.1, S4.1
- net N$11: now also BT-IO.2; no longer J3.2
- net N$12: now also BT-IO.3; no longer J3.3
- net N$2: now also BT-IO.1; no longer J3.1
Other:
- note added: "LED"
Changed lines of the file:
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@@
 <part name="S3" library="SparkFun-Switches" library_urn="urn:adsk.eagle:library:535" deviceset="MOMENTARY-SWITCH-SPST" device="-PTH-6.0MM" package3d_urn="urn:adsk.eagle:package:40163/1"/>
 <part name="S4" library="SparkFun-Switches" library_urn="urn:adsk.eagle:library:535" deviceset="MOMENTARY-SWITCH-SPST" device="-PTH-6.0MM" package3d_urn="urn:adsk.eagle:package:40163/1"/>
-<part name="J1" library="SparkFun-Connectors" library_urn="urn:adsk.eagle:library:513" deviceset="CONN_04" device="" package3d_urn="urn:adsk.eagle:package:38085/1"/>
-<part name="J3" library="SparkFun-Connectors" library_urn="urn:adsk.eagle:library:513" deviceset="CONN_03" device="" package3d_urn="urn:adsk.eagle:package:38063/1"/>
+<part name="OLED-IO" library="SparkFun-Connectors" library_urn="urn:adsk.eagle:library:513" deviceset="CONN_04" device="" package3d_urn="urn:adsk.eagle:package:38085/1"/>
+<part name="BT-IO" library="SparkFun-Connectors" library_urn="urn:adsk.eagle:library:513" deviceset="CONN_04" device="" package3d_urn="urn:adsk.eagle:package:38085/1"/>
+<part name="D1" library="SparkFun-LED" library_urn="urn:adsk.eagle:library:529" deviceset="LED" device="3MM" package3d_urn="urn:adsk.eagle:package:39361/1"/>
+<part name="R3-220" library="resistor" library_urn="urn:adsk.eagle:library:348" deviceset="R-EU_" device="R1206" package3d_urn="urn:adsk.eagle:package:26062/1" value="220"/>
 </parts>
 <sheets>
@@
 <text x="96.52" y="198.12" size="1.778" layer="91" rot="R90">GND</text>
 <text x="93.98" y="198.12" size="1.778" layer="91" rot="R90">5V</text>
-<text x="60.96" y="218.44" size="1.778" layer="91" rot="R90">D2</text>
-<text x="63.5" y="218.44" size="1.778" layer="91" rot="R90">D3</text>
-<text x="66.04" y="218.44" size="1.778" layer="91" rot="R90">D4</text>
+<text x="58.42" y="218.44" size="1.778" layer="91" rot="R90">D2</text>
+<text x="60.96" y="218.44" size="1.778" layer="91" rot="R90">D3</text>
+<text x="63.5" y="218.44" size="1.778" layer="91" rot="R90">D4</text>
+<text x="66.04" y="218.44" size="1.778" layer="91" rot="R90">LED</text>
 </plain>
 <instances>
@@
 <instance part="S3" gate="G$1" x="58.42" y="172.72" rot="R90"/>
 <instance part="S4" gate="G$1" x="53.34" y="175.26" rot="R90"/>
-<instance part="J1" gate="G$1" x="96.52" y="190.5" rot="R270"/>
-<instance part="J3" gate="J$1" x="60.96" y="213.36" rot="R270"/>
+<instance part="OLED-IO" gate="G$1" x="96.52" y="190.5" rot="R270"/>
+<instance part="BT-IO" gate="G$1" x="60.96" y="213.36" rot="R270"/>
+<instance part="D1" gate="G$1" x="86.36" y="220.98" rot="R270"/>
+<instance part="R3-220" gate="G$1" x="93.98" y="220.98" rot="R180"/>
 </instances>
 <busses>
@@
 </segment>
 </net>
-<net name="N$1" class="0">
+<net name="GND" class="0">
 <segment>
 <wire x1="99.06" y1="172.72" x2="99.06" y2="170.18" width="0.1524" layer="91"/>
@@
 <pinref part="IO3" gate="1" pin="1"/>
 <wire x1="99.06" y1="172.72" x2="96.52" y2="172.72" width="0.1524" layer="91"/>
-<wire x1="96.52" y1="172.72" x2="71.12" y2="172.72" width="0.1524" layer="91"/>
+<wire x1="96.52" y1="172.72" x2="76.2" y2="172.72" width="0.1524" layer="91"/>
+<wire x1="76.2" y1="172.72" x2="71.12" y2="172.72" width="0.1524" layer="91"/>
 <wire x1="116.84" y1="139.7" x2="114.3" y2="139.7" width="0.1524" layer="91"/>
 <wire x1="116.84" y1="139.7" x2="116.84" y2="170.18" width="0.1524" layer="91"/>
@@
 <wire x1="58.42" y1="165.1" x2="58.42" y2="167.64" width="0.1524" layer="91"/>
 <junction x="58.42" y="165.1"/>
-<pinref part="J1" gate="G$1" pin="2"/>
+<pinref part="OLED-IO" gate="G$1" pin="2"/>
 <wire x1="96.52" y1="185.42" x2="96.52" y2="172.72" width="0.1524" layer="91"/>
 <junction x="96.52" y="172.72"/>
+<pinref part="D1" gate="G$1" pin="C"/>
+<wire x1="81.28" y1="220.98" x2="76.2" y2="220.98" width="0.1524" layer="91"/>
+<wire x1="76.2" y1="220.98" x2="76.2" y2="172.72" width="0.1524" layer="91"/>
+<junction x="76.2" y="172.72"/>
 </segment>
 </net>
@@
 <wire x1="101.6" y1="172.72" x2="101.6" y2="175.26" width="0.1524" layer="91"/>
 <wire x1="101.6" y1="175.26" x2="93.98" y2="175.26" width="0.1524" layer="91"/>
-<pinref part="J1" gate="G$1" pin="1"/>
+<pinref part="OLED-IO" gate="G$1" pin="1"/>
 <wire x1="93.98" y1="185.42" x2="93.98" y2="175.26" width="0.1524" layer="91"/>
 </segment>
@@
 <wire x1="208.28" y1="172.72" x2="187.96" y2="152.4" width="0.1524" layer="91"/>
 <wire x1="187.96" y1="152.4" x2="81.28" y2="152.4" width="0.1524" layer="91"/>
-<pinref part="J1" gate="G$1" pin="4"/>
+<pinref part="OLED-IO" gate="G$1" pin="4"/>
 <wire x1="101.6" y1="185.42" x2="101.6" y2="182.88" width="0.1524" layer="91"/>
 <wire x1="101.6" y1="182.88" x2="81.28" y2="182.88" width="0.1524" layer="91"/>
@@
 <wire x1="205.74" y1="175.26" x2="185.42" y2="154.94" width="0.1524" layer="91"/>
 <wire x1="185.42" y1="154.94" x2="86.36" y2="154.94" width="0.1524" layer="91"/>
-<pinref part="J1" gate="G$1" pin="3"/>
+<pinref part="OLED-IO" gate="G$1" pin="3"/>
 <wire x1="99.06" y1="185.42" x2="99.06" y2="180.34" width="0.1524" layer="91"/>
 <wire x1="99.06" y1="180.34" x2="86.36" y2="180.34" width="0.1524" layer="91"/>
@@
 <segment>
 <pinref part="S4" gate="G$1" pin="2"/>
-<pinref part="J3" gate="J$1" pin="1"/>
+<pinref part="BT-IO" gate="G$1" pin="1"/>
 <wire x1="53.34" y1="180.34" x2="58.42" y2="180.34" width="0.1524" layer="91"/>
-<wire x1="58.42" y1="180.34" x2="58.42" y2="205.74" width="0.1524" layer="91"/>
+<wire x1="58.42" y1="180.34" x2="58.42" y2="208.28" width="0.1524" layer="91"/>
 </segment>
 </net>
@@
 <segment>
 <pinref part="S3" gate="G$1" pin="2"/>
-<pinref part="J3" gate="J$1" pin="2"/>
+<pinref part="BT-IO" gate="G$1" pin="2"/>
 <wire x1="58.42" y1="177.8" x2="60.96" y2="177.8" width="0.1524" layer="91"/>
-<wire x1="60.96" y1="177.8" x2="60.96" y2="205.74" width="0.1524" layer="91"/>
+<wire x1="60.96" y1="177.8" x2="60.96" y2="208.28" width="0.1524" layer="91"/>
 </segment>
 </net>
@@
 <segment>
 <pinref part="S2" gate="G$1" pin="2"/>
-<pinref part="J3" gate="J$1" pin="3"/>
-<wire x1="63.5" y1="175.26" x2="63.5" y2="205.74" width="0.1524" layer="91"/>
+<pinref part="BT-IO" gate="G$1" pin="3"/>
+<wire x1="63.5" y1="175.26" x2="63.5" y2="208.28" width="0.1524" layer="91"/>
 </segment>
 </net>
+<net name="N$1" class="0">
+<segment>
+<pinref part="D1" gate="G$1" pin="A"/>
+<pinref part="R3-220" gate="G$1" pin="2"/>
+</segment>
+</net>
+<net name="N$5" class="0">
+<segment>
+<pinref part="R3-220" gate="G$1" pin="1"/>
+<wire x1="104.14" y1="220.98" x2="99.06" y2="220.98" width="0.1524" layer="91"/>
+<wire x1="104.14" y1="213.36" x2="104.14" y2="220.98" width="0.1524" layer="91"/>
+<wire x1="86.36" y1="213.36" x2="104.14" y2="213.36" width="0.1524" layer="91"/>
+<wire x1="86.36" y1="205.74" x2="86.36" y2="213.36" width="0.1524" layer="91"/>
+<pinref part="BT-IO" gate="G$1" pin="4"/>
+<wire x1="66.04" y1="208.28" x2="66.04" y2="205.74" width="0.1524" layer="91"/>
+<wire x1="66.04" y1="205.74" x2="86.36" y2="205.74" width="0.1524" layer="91"/>
+</segment>
+</net>
