File: eagle/PCB/Module-PCB.brd (EAGLE design)
At the start: 35.6 x 27.9 mm, 10 parts

Commit message: Update PCB components
Other:
- board text added: "Pocket Groundstation"
- board text removed: "Pocket Groundsstation"
Changed lines of the file:
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@@
 <drawing>
 <settings>
-<setting alwaysvectorfont="yes"/>
+<setting alwaysvectorfont="no"/>
 <setting verticaltext="up"/>
 </settings>
@@
 <dimension x1="-41.91" y1="27.94" x2="-6.35" y2="29.21" x3="-24.13" y3="30.48" textsize="1.778" layer="1" dtype="horizontal"/>
 <dimension x1="-6.35" y1="27.94" x2="-6.35" y2="0" x3="-1.27" y3="13.97" textsize="1.778" layer="1" dtype="horizontal"/>
-<text x="-38.227" y="1.397" size="1.651" layer="25" rot="R90">Pocket Groundsstation</text>
+<text x="-38.227" y="1.397" size="1.651" layer="25" rot="R90">Pocket Groundstation</text>
 <text x="-17.78" y="6.35" size="1.778" layer="26" rot="MR90">MODULE SIDE</text>
 <text x="-35.687" y="1.397" size="1.651" layer="25" rot="R90">MODULE PCB | REV1</text>

Commit message: PCB updates
Parts:
- renumbered G to GND
Connections:
- net N$7 renamed GND
Routing:
- added copper zone on layer 1, net GND
- added copper zone on layer 16, net GND
