File: eagle/PCB/PCB 1c.brd (EAGLE design)
At the start: 45 x 75 mm, 27 parts

Commit message: update
Parts:
- moved AUD 3.81 mm to (10.2, 53.3)
- moved SER 3.81 mm to (10.2, 49.5)
Connections:
- net D10RX renamed D11-RX
- net HP5 renamed BUTTON1
- net HP6 renamed BUTTON3
- net N$1 renamed BUTTON2
- net N$10 renamed BUZZER
- net N$12 renamed VSENS
- net N$2 renamed 5V-OLED
- net N$4 renamed BEC-5V
- net N$7 renamed LED
Changed lines of the file:
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@@
 <layer number="19" name="Unrouted" color="6" fill="1" visible="yes" active="yes"/>
 <layer number="20" name="Dimension" color="24" fill="1" visible="yes" active="yes"/>
-<layer number="21" name="tPlace" color="7" fill="1" visible="yes" active="yes"/>
+<layer number="21" name="tPlace" color="7" fill="1" visible="no" active="yes"/>
 <layer number="22" name="bPlace" color="7" fill="1" visible="yes" active="yes"/>
-<layer number="23" name="tOrigins" color="15" fill="1" visible="yes" active="yes"/>
+<layer number="23" name="tOrigins" color="15" fill="1" visible="no" active="yes"/>
 <layer number="24" name="bOrigins" color="15" fill="1" visible="yes" active="yes"/>
-<layer number="25" name="tNames" color="7" fill="1" visible="yes" active="yes"/>
+<layer number="25" name="tNames" color="7" fill="1" visible="no" active="yes"/>
 <layer number="26" name="bNames" color="7" fill="1" visible="yes" active="yes"/>
 <layer number="27" name="tValues" color="7" fill="1" visible="no" active="yes"/>
@@
 <layer number="37" name="tTest" color="7" fill="1" visible="no" active="yes"/>
 <layer number="38" name="bTest" color="7" fill="1" visible="no" active="yes"/>
-<layer number="39" name="tKeepout" color="4" fill="11" visible="yes" active="yes"/>
+<layer number="39" name="tKeepout" color="4" fill="11" visible="no" active="yes"/>
 <layer number="40" name="bKeepout" color="1" fill="11" visible="yes" active="yes"/>
-<layer number="41" name="tRestrict" color="4" fill="10" visible="yes" active="yes"/>
+<layer number="41" name="tRestrict" color="4" fill="10" visible="no" active="yes"/>
 <layer number="42" name="bRestrict" color="1" fill="10" visible="yes" active="yes"/>
 <layer number="43" name="vRestrict" color="2" fill="10" visible="no" active="yes"/>
@@
 <layer number="49" name="Reference" color="7" fill="1" visible="no" active="yes"/>
 <layer number="50" name="dxf" color="7" fill="1" visible="no" active="no"/>
-<layer number="51" name="tDocu" color="7" fill="1" visible="yes" active="yes"/>
+<layer number="51" name="tDocu" color="7" fill="1" visible="no" active="yes"/>
 <layer number="52" name="bDocu" color="7" fill="1" visible="yes" active="yes"/>
 <layer number="53" name="tGND_GNDA" color="7" fill="9" visible="no" active="no"/>
@@
 <attribute name="VALUE" x="43.18" y="40.259" size="0.6096" layer="27" font="vector" ratio="20" rot="R90"/>
 </element>
-<element name="SER" library="SparkFun-Connectors" library_urn="urn:adsk.eagle:library:513" package="1X01" package3d_urn="urn:adsk.eagle:package:38028/1" value="" x="10.16" y="53.34" rot="MR90"/>
-<element name="AUD" library="SparkFun-Connectors" library_urn="urn:adsk.eagle:library:513" package="1X01" package3d_urn="urn:adsk.eagle:package:38028/1" value="" x="10.16" y="49.53" rot="MR90"/>
+<element name="SER" library="SparkFun-Connectors" library_urn="urn:adsk.eagle:library:513" package="1X01" package3d_urn="urn:adsk.eagle:package:38028/1" value="" x="10.16" y="49.53" rot="MR90"/>
+<element name="AUD" library="SparkFun-Connectors" library_urn="urn:adsk.eagle:library:513" package="1X01" package3d_urn="urn:adsk.eagle:package:38028/1" value="" x="10.16" y="53.34" rot="MR90"/>
 <element name="M_0446200001" library="con-molex" library_urn="urn:adsk.eagle:library:165" package="0446200001" value="0446200001" x="15.0876" y="71.9836" smashed="yes" rot="R180">
 <attribute name="MF" value="MOLEX" x="15.0876" y="71.9836" size="1.778" layer="27" rot="R180" display="off"/>
@@
 </elements>
 <signals>
-<signal name="N$2">
+<signal name="5V-OLED">
 <contactref element="U$1" pad="VCC"/>
 <contactref element="OLED" pad="4"/>
@@
 <wire x1="40.64" y1="43.37" x2="30.48" y2="53.34" width="0" layer="19" extent="1-1"/>
 </signal>
-<signal name="D10RX" class="1">
+<signal name="D11-RX" class="1">
 <contactref element="U$1" pad="D11"/>
 <contactref element="J3" pad="1"/>
@@
 <wire x1="3.81" y1="55.88" x2="20.32" y2="57.785" width="0" layer="19" extent="1-1"/>
 </signal>
-<signal name="HP5" class="1">
+<signal name="BUTTON1" class="1">
 <contactref element="U$1" pad="D2"/>
 <contactref element="BT-BRIDGE" pad="3"/>
 <wire x1="25.4" y1="2.54" x2="21.59" y2="20.32" width="0" layer="19" extent="1-1"/>
 </signal>
-<signal name="HP6" class="1">
+<signal name="BUTTON3" class="1">
 <contactref element="BT-BRIDGE" pad="1"/>
 <contactref element="U$1" pad="D4"/>
 <wire x1="30.48" y1="2.54" x2="26.67" y2="20.32" width="0" layer="19" extent="1-1"/>
 </signal>
-<signal name="N$10" class="1">
+<signal name="BUZZER" class="1">
 <contactref element="BUZZ" pad="+"/>
 <contactref element="U$1" pad="D9"/>
@@
 <contactref element="MINIMOSD" pad="BGND"/>
 </signal>
-<signal name="N$12">
+<signal name="VSENS">
 <contactref element="R1-18K" pad="1"/>
 <contactref element="R2-4.7K" pad="2"/>
@@
 <wire x1="3.81" y1="36.83" x2="29.21" y2="20.32" width="0" layer="19" extent="1-1"/>
 </signal>
-<signal name="N$1" class="1">
+<signal name="BUTTON2" class="1">
 <contactref element="U$1" pad="D3"/>
 <contactref element="BT-BRIDGE" pad="2"/>
 <wire x1="27.94" y1="2.54" x2="24.13" y2="20.32" width="0" layer="19" extent="1-1"/>
 </signal>
-<signal name="N$4">
+<signal name="BEC-5V">
 <contactref element="U$1" pad="RAW"/>
 <contactref element="D1" pad="K"/>
@@
 <wire x1="33.73" y1="64.73" x2="33.73" y2="68.73" width="0" layer="19" extent="1-1"/>
 <wire x1="15.5956" y1="69.4436" x2="33.73" y2="68.73" width="0" layer="19" extent="1-1"/>
-<wire x1="10.16" y1="49.53" x2="15.5956" y2="69.4436" width="0" layer="19" extent="1-1"/>
+<wire x1="10.16" y1="53.34" x2="15.5956" y2="69.4436" width="0" layer="19" extent="1-1"/>
 </signal>
 <signal name="VMAIN" class="2">
@@
 <wire x1="3.81" y1="58.42" x2="13.5636" y2="69.4436" width="0" layer="19" extent="1-1"/>
 </signal>
-<signal name="N$7" class="1">
+<signal name="LED" class="1">
 <contactref element="U$1" pad="D13"/>
 <contactref element="BT-BRIDGE" pad="4"/>
