File: eagle/PCB/PCB 1c.brd (EAGLE design)
At the start: 45 x 75 mm, 27 parts

Commit message: Component change
Parts:
- removed BUZZ: BUZZER-PTH, SparkFun-Electromechanical:BUZZER-12MM
- added SG1: F/TMB, buzzer:F/TMB
Connections:
- net BUZZER: now also SG1.+; no longer BUZZ.+
- net GND: now also SG1.-; no longer BUZZ.-
Changed lines of the file:
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@@
 <drawing>
 <settings>
-<setting alwaysvectorfont="yes"/>
+<setting alwaysvectorfont="no"/>
 <setting verticaltext="up"/>
 </settings>
@@
 <attribute name="VALUE" x="15.24" y="3.54" size="0.0254" layer="27"/>
 </element>
-<element name="BUZZ" library="SparkFun-Electromechanical" library_urn="urn:adsk.eagle:library:516" package="BUZZER-12MM" package3d_urn="urn:adsk.eagle:package:38558/1" value="BUZZER-PTH" x="38.1" y="7.62" smashed="yes" rot="R90">
-<attribute name="NAME" x="36.195" y="5.08" size="1.27" layer="25" ratio="10" rot="R90"/>
-<attribute name="PROD_ID" value="COMP-08253" x="38.1" y="7.62" size="1.778" layer="27" rot="R90" display="off"/>
-<attribute name="SF_SKU" value="COM-07950" x="38.1" y="7.62" size="1.778" layer="27" rot="R90" display="off"/>
-<attribute name="SPICEPREFIX" value="X" x="38.1" y="7.62" size="1.778" layer="27" rot="R90" display="off"/>
-<attribute name="VALUE" x="41.91" y="3.175" size="1.27" layer="27" ratio="10" rot="R90"/>
-</element>
 <element name="MINIMOSD" library="FPVTools" package="MMOSDNVDVID" value="MICROMINIMOSDPWR" x="22.86" y="49.53"/>
 <element name="R1-18K" library="rcl" library_urn="urn:adsk.eagle:library:334" package="M1206" package3d_urn="urn:adsk.eagle:package:23566/1" value="18k Ohm" x="16.51" y="27.94" smashed="yes" rot="R180">
@@
 <attribute name="VALUE" x="31.496" y="17.653" size="0.0254" layer="27" rot="R180"/>
 </element>
+<element name="SG1" library="buzzer" library_urn="urn:adsk.eagle:library:113" package="F/TMB" package3d_urn="urn:adsk.eagle:package:5260/1" value="F/TMB" x="38.1" y="7.62">
+<attribute name="MF" value="" x="38.1" y="7.62" size="1.778" layer="27" display="off"/>
+<attribute name="MPN" value="" x="38.1" y="7.62" size="1.778" layer="27" display="off"/>
+<attribute name="OC_FARNELL" value="unknown" x="38.1" y="7.62" size="1.778" layer="27" display="off"/>
+<attribute name="OC_NEWARK" value="unknown" x="38.1" y="7.62" size="1.778" layer="27" display="off"/>
+</element>
 </elements>
 <signals>
@@
 <contactref element="MINIMOSD" pad="IGND"/>
 <contactref element="DVR/MODULE-IO" pad="3"/>
-<contactref element="BUZZ" pad="-"/>
 <contactref element="U$1" pad="GND"/>
 <contactref element="OLED" pad="3"/>
@@
 <contactref element="M_0446200001" pad="4"/>
 <contactref element="M_0446200001" pad="2"/>
+<contactref element="SG1" pad="-"/>
 <wire x1="33.73" y1="71.73" x2="39.37" y2="66.04" width="0" layer="19" extent="1-1"/>
 <wire x1="41.91" y1="57.15" x2="39.37" y2="66.04" width="0" layer="19" extent="1-1"/>
@@
 <wire x1="28.07" y1="27.94" x2="25.4" y2="40.6" width="0" layer="19" extent="1-1"/>
 <wire x1="30.48" y1="16.51" x2="28.07" y2="27.94" width="0" layer="19" extent="1-1"/>
-<wire x1="38.1" y1="4.37" x2="30.48" y2="16.51" width="0" layer="19" extent="1-1"/>
+<wire x1="34.29" y1="7.62" x2="30.48" y2="16.51" width="0" layer="19" extent="1-1"/>
 <wire x1="15.24" y1="16.51" x2="30.48" y2="16.51" width="0" layer="19" extent="1-1"/>
 <wire x1="12.42" y1="8.89" x2="15.24" y2="16.51" width="0" layer="19" extent="1-1"/>
@@
 </signal>
 <signal name="BUZZER" class="1">
-<contactref element="BUZZ" pad="+"/>
 <contactref element="U$1" pad="D9"/>
-<wire x1="38.1" y1="10.87" x2="39.37" y2="20.32" width="0" layer="19" extent="1-1"/>
+<contactref element="SG1" pad="+"/>
+<wire x1="41.91" y1="7.62" x2="39.37" y2="20.32" width="0" layer="19" extent="1-1"/>
 </signal>
 <signal name="DVRVIDEO-IN" class="2">

Commit message: PCB Updates
Routing:
- net +5V: track 0.00 -> 87.5 mm, vias 0 -> 4
- net VCC: track 0.00 -> 68.5 mm, vias 0 -> 2
- net SCL: track 0.00 -> 54.7 mm
- net AUDIO: track 0.00 -> 53.1 mm, vias 0 -> 2
- net LED: track 0.00 -> 50.2 mm
- net D6: track 0.00 -> 49.4 mm, vias 0 -> 1
- net SDA: track 0.00 -> 46.8 mm
- net D7: track 0.00 -> 44.4 mm
- net BEC-5V: track 0.00 -> 44.0 mm, vias 0 -> 1
- net D5: track 0.00 -> 39.7 mm
- net VMAIN: track 0.00 -> 39.0 mm
- net 5V-OLED: track 0.00 -> 38.1 mm
- net RAWVIDEO_MODULE: track 0.00 -> 29.2 mm
- net 8V: track 0.00 -> 24.1 mm
- net BUTTON3: track 0.00 -> 19.4 mm
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- added copper zone on layer 1, net GND
- added copper zone on layer 16, net GND

Commit message: PCB Updates
Connections:
- removed net 5V-OLED: OLED.4, U$1.VCC
- net BEC-5V: now also OLED.4, U$1.VCC; no longer U$1.RAW
Routing:
- net 5V-OLED: track 38.1 -> 0.00 mm
- net BEC-5V: track 44.0 -> 74.7 mm
Changed lines of the file:
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@@
 <text x="2.54" y="19.05" size="1.016" layer="26" rot="MR90">&lt; To switch</text>
 <text x="12.7" y="1.27" size="1.016" layer="26" rot="MR0">&lt; From switch</text>
-<text x="43.18" y="36.83" size="1.27" layer="26" rot="MR270">POCKET-GROUNDSTATION | PCB1 | REV1</text>
+<text x="43.18" y="48.26" size="1.27" layer="26" rot="MR270">POCKET-GROUNDSTATION | PCB1 | REV1</text>
 <text x="1.27" y="48.26" size="0.889" layer="26" rot="MR90">Vout</text>
 <text x="6.35" y="53.34" size="0.889" layer="26" rot="MR0">VIN/DVR</text>
@@
 </elements>
 <signals>
-<signal name="5V-OLED">
-<contactref element="U$1" pad="VCC"/>
-<contactref element="OLED" pad="4"/>
-<wire x1="20.0025" y1="36.5125" x2="19.05" y2="35.56" width="0.762" layer="16"/>
-<wire x1="20.0025" y1="36.83" x2="20.0025" y2="36.5125" width="0.762" layer="16"/>
-<wire x1="21.2725" y1="38.1" x2="20.0025" y2="36.83" width="0.762" layer="16"/>
-<wire x1="28.575" y1="38.1" x2="21.2725" y2="38.1" width="0.762" layer="16"/>
-<wire x1="33.655" y1="43.18" x2="28.575" y2="38.1" width="0.762" layer="16"/>
-<wire x1="33.655" y1="51.7525" x2="33.655" y2="43.18" width="0.762" layer="16"/>
-<wire x1="41.5925" y1="59.69" x2="33.655" y2="51.7525" width="0.762" layer="16"/>
-<wire x1="41.91" y1="59.69" x2="41.5925" y2="59.69" width="0.762" layer="16"/>
-</signal>
 <signal name="SCL" class="1">
 <contactref element="U$1" pad="A5"/>
@@
 <vertex x="-2.54" y="-2.54"/>
 </polygon>
+<wire x1="13.6525" y1="8.255" x2="13.750196875" y2="8.255" width="0.762" layer="1"/>
 <wire x1="12.42" y1="8.89" x2="15.24" y2="16.51" width="0" layer="19" extent="1-1"/>
 </signal>
@@
 </signal>
 <signal name="BEC-5V">
-<contactref element="U$1" pad="RAW"/>
 <contactref element="D1" pad="K"/>
 <wire x1="39.6875" y1="15.875" x2="39.0525" y2="15.24" width="0.762" layer="1"/>
@@
 <wire x1="29.845" y1="26.9875" x2="35.56" y2="26.9875" width="0.762" layer="1"/>
 <wire x1="23.495" y1="33.3375" x2="29.845" y2="26.9875" width="0.762" layer="16"/>
-<wire x1="13.335" y1="33.3375" x2="23.495" y2="33.3375" width="0.762" layer="16"/>
-<wire x1="11.43" y1="35.2425" x2="13.335" y2="33.3375" width="0.762" layer="16"/>
-<wire x1="11.43" y1="35.56" x2="11.43" y2="35.2425" width="0.762" layer="16"/>
 <wire x1="39.0525" y1="15.24" x2="38.88" y2="15.24" width="0.762" layer="1"/>
 <via x="29.845" y="26.9875" extent="1-16" drill="0.508"/>
+<contactref element="U$1" pad="VCC"/>
+<contactref element="OLED" pad="4"/>
+<wire x1="20.0025" y1="36.5125" x2="19.05" y2="35.56" width="0.762" layer="16"/>
+<wire x1="20.0025" y1="36.83" x2="20.0025" y2="36.5125" width="0.762" layer="16"/>
+<wire x1="21.2725" y1="38.1" x2="20.0025" y2="36.83" width="0.762" layer="16"/>
+<wire x1="28.575" y1="38.1" x2="21.2725" y2="38.1" width="0.762" layer="16"/>
+<wire x1="33.655" y1="43.18" x2="28.575" y2="38.1" width="0.762" layer="16"/>
+<wire x1="33.655" y1="51.7525" x2="33.655" y2="43.18" width="0.762" layer="16"/>
+<wire x1="41.5925" y1="59.69" x2="33.655" y2="51.7525" width="0.762" layer="16"/>
+<wire x1="41.91" y1="59.69" x2="41.5925" y2="59.69" width="0.762" layer="16"/>
+<wire x1="20.955" y1="33.3375" x2="23.495" y2="33.3375" width="0.762" layer="16"/>
+<wire x1="19.3675" y1="34.925" x2="20.955" y2="33.3375" width="0.762" layer="16"/>
+<wire x1="19.05" y1="34.925" x2="19.3675" y2="34.925" width="0.762" layer="16"/>
+<wire x1="19.05" y1="34.925" x2="19.05" y2="35.56" width="0.762" layer="16"/>
 </signal>
 <signal name="RX" class="1">

Commit message: pcb updates
Parts:
- added A1: TPTP20SQ, testpad:TP20SQ
Connections:
- new net N$1: A1.TP, U$1.A1
Routing:
- net N$1: track 0.00 -> 5.76 mm
Changed lines of the file:
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@@
 <drawing>
 <settings>
-<setting alwaysvectorfont="yes"/>
+<setting alwaysvectorfont="no"/>
 <setting verticaltext="up"/>
 </settings>
@@
 <attribute name="OC_NEWARK" value="unknown" x="38.1" y="7.62" size="1.778" layer="27" display="off"/>
 </element>
+<element name="A1" library="testpad" library_urn="urn:adsk.eagle:library:385" package="TP20SQ" package3d_urn="urn:adsk.eagle:package:27980/1" value="TPTP20SQ" x="30.48" y="31.75" rot="MR90">
+<attribute name="TP_SIGNAL_NAME" value="" x="30.48" y="31.75" size="1.778" layer="28" rot="MR90" display="off"/>
+</element>
 </elements>
 <signals>
@@
 <wire x1="34.29" y1="39.37" x2="30.48" y2="43.18" width="0.381" layer="1"/>
 </signal>
+<signal name="N$1">
+<contactref element="A1" pad="TP"/>
+<contactref element="U$1" pad="A1"/>
+<wire x1="29.21" y1="33.02" x2="30.48" y2="31.75" width="0.762" layer="16"/>
+<wire x1="28.575" y1="33.02" x2="29.21" y2="33.02" width="0.762" layer="16"/>
+<wire x1="26.67" y1="34.925" x2="28.575" y2="33.02" width="0.762" layer="16"/>
+<wire x1="26.67" y1="35.56" x2="26.67" y2="34.925" width="0.762" layer="16"/>
+</signal>
 </signals>

Commit message: PCB change
Connections:
- net GND: now also PJ-320D.EARTH; no longer PJ-320D.RING2
- net VMAIN: now also PJ-320D.RING2; no longer PJ-320D.EARTH
Routing:
- net VMAIN: track 39.0 -> 45.4 mm
- net AUDIO: track 53.1 -> 47.0 mm, vias 2 -> 3
Changed lines of the file:
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@@
 <drawing>
 <settings>
-<setting alwaysvectorfont="no"/>
+<setting alwaysvectorfont="yes"/>
 <setting verticaltext="up"/>
 </settings>
@@
 <layer number="14" name="Route14" color="1" fill="6" visible="no" active="no"/>
 <layer number="15" name="Route15" color="4" fill="6" visible="no" active="no"/>
-<layer number="16" name="Bottom" color="1" fill="1" visible="yes" active="yes"/>
+<layer number="16" name="Bottom" color="1" fill="1" visible="no" active="yes"/>
 <layer number="17" name="Pads" color="2" fill="1" visible="yes" active="yes"/>
 <layer number="18" name="Vias" color="2" fill="1" visible="yes" active="yes"/>
@@
 <layer number="20" name="Dimension" color="24" fill="1" visible="yes" active="yes"/>
 <layer number="21" name="tPlace" color="7" fill="1" visible="yes" active="yes"/>
-<layer number="22" name="bPlace" color="7" fill="1" visible="yes" active="yes"/>
+<layer number="22" name="bPlace" color="7" fill="1" visible="no" active="yes"/>
 <layer number="23" name="tOrigins" color="15" fill="1" visible="yes" active="yes"/>
-<layer number="24" name="bOrigins" color="15" fill="1" visible="yes" active="yes"/>
+<layer number="24" name="bOrigins" color="15" fill="1" visible="no" active="yes"/>
 <layer number="25" name="tNames" color="7" fill="1" visible="yes" active="yes"/>
-<layer number="26" name="bNames" color="7" fill="1" visible="yes" active="yes"/>
+<layer number="26" name="bNames" color="7" fill="1" visible="no" active="yes"/>
 <layer number="27" name="tValues" color="7" fill="1" visible="no" active="yes"/>
 <layer number="28" name="bValues" color="7" fill="1" visible="no" active="yes"/>
@@
 <layer number="38" name="bTest" color="7" fill="1" visible="no" active="yes"/>
 <layer number="39" name="tKeepout" color="4" fill="11" visible="yes" active="yes"/>
-<layer number="40" name="bKeepout" color="1" fill="11" visible="yes" active="yes"/>
+<layer number="40" name="bKeepout" color="1" fill="11" visible="no" active="yes"/>
 <layer number="41" name="tRestrict" color="4" fill="10" visible="yes" active="yes"/>
-<layer number="42" name="bRestrict" color="1" fill="10" visible="yes" active="yes"/>
+<layer number="42" name="bRestrict" color="1" fill="10" visible="no" active="yes"/>
 <layer number="43" name="vRestrict" color="2" fill="10" visible="no" active="yes"/>
 <layer number="44" name="Drills" color="7" fill="1" visible="no" active="yes"/>
@@
 <layer number="50" name="dxf" color="7" fill="1" visible="no" active="no"/>
 <layer number="51" name="tDocu" color="7" fill="1" visible="yes" active="yes"/>
-<layer number="52" name="bDocu" color="7" fill="1" visible="yes" active="yes"/>
+<layer number="52" name="bDocu" color="7" fill="1" visible="no" active="yes"/>
 <layer number="53" name="tGND_GNDA" color="7" fill="9" visible="no" active="no"/>
 <layer number="54" name="bGND_GNDA" color="1" fill="9" visible="no" active="no"/>
@@
 <contactref element="R2-4.7K" pad="1"/>
 <contactref element="MINIMOSD" pad="VGND2"/>
-<contactref element="PJ-320D" pad="RING2"/>
 <contactref element="IN-" pad="TP"/>
 <contactref element="-OUT" pad="TP"/>
@@
 </polygon>
 <wire x1="13.6525" y1="8.255" x2="13.750196875" y2="8.255" width="0.762" layer="1"/>
+<contactref element="PJ-320D" pad="EARTH"/>
+<wire x1="40.9575" y1="57.785" x2="40.855428125" y2="57.859159375" width="0.762" layer="1"/>
 <wire x1="12.42" y1="8.89" x2="15.24" y2="16.51" width="0" layer="19" extent="1-1"/>
 </signal>
@@
 <wire x1="18.0975" y1="71.12" x2="17.145" y2="71.12" width="0.5" layer="16"/>
 <wire x1="20.32" y1="68.8975" x2="18.0975" y2="71.12" width="0.5" layer="16"/>
-<wire x1="28.2575" y1="68.8975" x2="20.32" y2="68.8975" width="0.5" layer="16"/>
+<wire x1="28.2575" y1="68.8975" x2="25.0825" y2="68.8975" width="0.5" layer="16"/>
+<wire x1="25.0825" y1="68.8975" x2="20.32" y2="68.8975" width="0.5" layer="16"/>
 <wire x1="33.655" y1="68.8975" x2="28.2575" y2="68.8975" width="0.5" layer="1"/>
 <wire x1="15.875" y1="69.5325" x2="15.5956" y2="69.4436" width="0.5" layer="16"/>
@@
 <wire x1="10.16" y1="53.975" x2="10.16" y2="53.34" width="0.5" layer="16"/>
 <wire x1="18.0975" y1="61.9125" x2="10.16" y2="53.975" width="0.5" layer="16"/>
-<wire x1="31.115" y1="61.9125" x2="18.0975" y2="61.9125" width="0.5" layer="1"/>
-<wire x1="33.655" y1="64.4525" x2="31.115" y2="61.9125" width="0.5" layer="1"/>
 <wire x1="33.655" y1="64.4525" x2="33.73" y2="64.73" width="0.5" layer="1"/>
 <via x="28.2575" y="68.8975" extent="1-16" drill="0.4"/>
 <via x="18.0975" y="61.9125" extent="1-16" drill="0.4"/>
+<wire x1="25.0825" y1="68.8975" x2="18.0975" y2="61.9125" width="0.5" layer="1"/>
+<wire x1="25.0825" y1="69.215" x2="25.0825" y2="68.8975" width="0.5" layer="1"/>
+<wire x1="25.0825" y1="68.8975" x2="25.0825" y2="69.215" width="0.5" layer="16"/>
+<via x="25.0825" y="69.215" extent="1-16" drill="0.4"/>
 </signal>
 <signal name="VMAIN" class="2">
 <contactref element="V-IO" pad="3"/>
-<contactref element="PJ-320D" pad="EARTH"/>
 <contactref element="M_0446200001" pad="3"/>
-<wire x1="25.4" y1="63.8175" x2="26.9875" y2="63.8175" width="0.5" layer="1"/>
 <wire x1="18.0975" y1="71.12" x2="21.43125" y2="67.78625" width="0.5" layer="1"/>
-<wire x1="21.43125" y1="67.78625" x2="25.4" y2="63.8175" width="0.5" layer="1"/>
 <wire x1="15.24" y1="71.12" x2="18.0975" y2="71.12" width="0.5" layer="1"/>
 <wire x1="13.5636" y1="69.4436" x2="15.24" y2="71.12" width="0.5" layer="1"/>
-<wire x1="26.9875" y1="63.8175" x2="27.23" y2="63.63" width="0.5" layer="1"/>
 <wire x1="12.065" y1="58.42" x2="3.81" y2="58.42" width="0.5" layer="1"/>
 <wire x1="21.43125" y1="67.78625" x2="12.065" y2="58.42" width="0.5" layer="1"/>
+<contactref element="PJ-320D" pad="RING2"/>
+<wire x1="31.75" y1="71.4375" x2="33.655" y2="71.4375" width="0.5" layer="1"/>
+<wire x1="30.7975" y1="70.485" x2="31.75" y2="71.4375" width="0.5" layer="1"/>
+<wire x1="25.0825" y1="70.485" x2="30.7975" y2="70.485" width="0.5" layer="1"/>
+<wire x1="24.4475" y1="70.1675" x2="25.0825" y2="70.485" width="0.5" layer="1"/>
+<wire x1="22.225" y1="67.945" x2="24.4475" y2="70.1675" width="0.5" layer="1"/>
+<wire x1="21.59" y1="67.945" x2="22.225" y2="67.945" width="0.5" layer="1"/>
+<wire x1="33.655" y1="71.4375" x2="33.73" y2="71.73" width="0.5" layer="1"/>
+<wire x1="21.59" y1="67.945" x2="21.43125" y2="67.78625" width="0.5" layer="1"/>
 </signal>
 <signal name="LED" class="1">
