File: eagle/PCB/PCB 2c.brd (EAGLE design)
At the start: 45 x 75 mm, 14 parts

Commit message: PCB Updates
Routing:
- net N$5: track 0.00 -> 62.7 mm
- net N$4: track 0.00 -> 23.5 mm
- net N$7: track 0.00 -> 21.4 mm
- net N$6: track 0.00 -> 20.8 mm
- net N$10: track 0.00 -> 19.9 mm
- net N$12: track 0.00 -> 17.2 mm
- net N$3: track 0.00 -> 15.7 mm
- net N$11: track 0.00 -> 15.1 mm
- net N$2: track 0.00 -> 14.3 mm
- net VIDOUT: track 0.00 -> 13.3 mm
- net N$1: track 0.00 -> 3.92 mm
- added copper zone on layer 1, net GND
- added copper zone on layer 16, net GND
Changed lines of the file:
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@@
 <drawing>
 <settings>
-<setting alwaysvectorfont="no"/>
+<setting alwaysvectorfont="yes"/>
 <setting verticaltext="up"/>
 </settings>
@@
 <contactref element="IO3" pad="4"/>
 <contactref element="S1" pad="1"/>
-<wire x1="3.81" y1="55.88" x2="13.97" y2="63.5" width="0" layer="19" extent="1-1"/>
+<wire x1="5.3975" y1="55.88" x2="3.81" y2="55.88" width="0.4" layer="16"/>
+<wire x1="12.3825" y1="62.865" x2="5.3975" y2="55.88" width="0.4" layer="16"/>
+<wire x1="12.7" y1="62.865" x2="12.3825" y2="62.865" width="0.4" layer="16"/>
+<wire x1="13.335" y1="63.5" x2="12.7" y2="62.865" width="0.4" layer="16"/>
+<wire x1="13.97" y1="63.5" x2="13.335" y2="63.5" width="0.4" layer="16"/>
 </signal>
 <signal name="N$3" class="2">
 <contactref element="IO3" pad="3"/>
 <contactref element="S1" pad="2"/>
-<wire x1="3.81" y1="58.42" x2="16.51" y2="63.5" width="0" layer="19" extent="1-1"/>
+<wire x1="5.3975" y1="58.42" x2="3.81" y2="58.42" width="0.4" layer="1"/>
+<wire x1="7.3025" y1="60.325" x2="5.3975" y2="58.42" width="0.4" layer="1"/>
+<wire x1="14.9225" y1="60.325" x2="7.3025" y2="60.325" width="0.4" layer="1"/>
+<wire x1="16.51" y1="61.9125" x2="14.9225" y2="60.325" width="0.4" layer="1"/>
+<wire x1="16.51" y1="63.5" x2="16.51" y2="61.9125" width="0.4" layer="1"/>
 </signal>
 <signal name="GND">
@@
 <contactref element="OLED-IO" pad="2"/>
 <contactref element="D1" pad="K"/>
-<wire x1="33.02" y1="63.5" x2="41.91" y2="57.15" width="0" layer="19" extent="1-1"/>
-<wire x1="36.83" y1="41.91" x2="41.91" y2="57.15" width="0" layer="19" extent="1-1"/>
-<wire x1="35.0012" y1="10.4394" x2="36.83" y2="41.91" width="0" layer="19" extent="1-1"/>
-<wire x1="26.1112" y1="10.4394" x2="35.0012" y2="10.4394" width="0" layer="19" extent="1-1"/>
-<wire x1="17.2212" y1="10.4394" x2="26.1112" y2="10.4394" width="0" layer="19" extent="1-1"/>
-<wire x1="3.81" y1="63.5" x2="33.02" y2="63.5" width="0" layer="19" extent="1-1"/>
+<polygon width="0.1524" layer="1">
+<vertex x="0" y="74.93"/>
+<vertex x="0" y="-1.27"/>
+<vertex x="45.72" y="-1.27"/>
+<vertex x="45.72" y="76.2"/>
+<vertex x="0" y="76.2"/>
+</polygon>
+<polygon width="0.1524" layer="16">
+<vertex x="-1.27" y="76.2"/>
+<vertex x="46.99" y="76.2"/>
+<vertex x="46.99" y="-2.54"/>
+<vertex x="-1.27" y="-2.54"/>
+</polygon>
 </signal>
 <signal name="N$4">
 <contactref element="OLED" pad="2"/>
 <contactref element="OLED-IO" pad="1"/>
-<wire x1="36.83" y1="39.37" x2="41.91" y2="59.69" width="0" layer="19" extent="1-1"/>
+<wire x1="38.1" y1="39.37" x2="36.83" y2="39.37" width="0.762" layer="16"/>
+<wire x1="39.37" y1="40.64" x2="38.1" y2="39.37" width="0.762" layer="16"/>
+<wire x1="39.37" y1="57.785" x2="39.37" y2="40.64" width="0.762" layer="16"/>
+<wire x1="41.275" y1="59.69" x2="39.37" y2="57.785" width="0.762" layer="16"/>
+<wire x1="41.91" y1="59.69" x2="41.275" y2="59.69" width="0.762" layer="16"/>
 </signal>
 <signal name="N$6" class="1">
 <contactref element="OLED-IO" pad="4"/>
 <contactref element="OLED" pad="4"/>
-<wire x1="36.83" y1="34.29" x2="41.91" y2="52.07" width="0" layer="19" extent="1-1"/>
+<wire x1="38.4175" y1="34.29" x2="36.83" y2="34.29" width="0.3" layer="1"/>
+<wire x1="40.9575" y1="36.83" x2="38.4175" y2="34.29" width="0.3" layer="1"/>
+<wire x1="40.9575" y1="50.4825" x2="40.9575" y2="36.83" width="0.3" layer="1"/>
+<wire x1="41.91" y1="51.435" x2="40.9575" y2="50.4825" width="0.3" layer="1"/>
+<wire x1="41.91" y1="52.07" x2="41.91" y2="51.435" width="0.3" layer="1"/>
 </signal>
 <signal name="N$7" class="1">
 <contactref element="OLED-IO" pad="3"/>
 <contactref element="OLED" pad="3"/>
-<wire x1="36.83" y1="36.83" x2="41.91" y2="54.61" width="0" layer="19" extent="1-1"/>
+<wire x1="38.4175" y1="36.83" x2="36.83" y2="36.83" width="0.3" layer="1"/>
+<wire x1="39.37" y1="37.7825" x2="38.4175" y2="36.83" width="0.3" layer="1"/>
+<wire x1="39.37" y1="53.0225" x2="39.37" y2="37.7825" width="0.3" layer="1"/>
+<wire x1="40.9575" y1="54.61" x2="39.37" y2="53.0225" width="0.3" layer="1"/>
+<wire x1="41.91" y1="54.61" x2="40.9575" y2="54.61" width="0.3" layer="1"/>
 </signal>
 <signal name="N$10" class="2">
 <contactref element="IO3" pad="2"/>
 <contactref element="S1" pad="3"/>
-<wire x1="3.81" y1="60.96" x2="19.05" y2="63.5" width="0" layer="19" extent="1-1"/>
+<wire x1="5.3975" y1="60.96" x2="3.81" y2="60.96" width="0.4" layer="1"/>
+<wire x1="11.1125" y1="66.675" x2="5.3975" y2="60.96" width="0.4" layer="1"/>
+<wire x1="17.4625" y1="66.675" x2="11.1125" y2="66.675" width="0.4" layer="1"/>
+<wire x1="19.05" y1="65.0875" x2="17.4625" y2="66.675" width="0.4" layer="1"/>
+<wire x1="19.05" y1="63.5" x2="19.05" y2="65.0875" width="0.4" layer="1"/>
 </signal>
 <signal name="N$2" class="1">
 <contactref element="S4" pad="3"/>
 <contactref element="BT-IO" pad="1"/>
-<wire x1="30.48" y1="2.54" x2="35.0012" y2="14.9606" width="0" layer="19" extent="1-1"/>
+<wire x1="32.7025" y1="4.7625" x2="30.48" y2="2.54" width="0.3" layer="1"/>
+<wire x1="32.7025" y1="12.7" x2="32.7025" y2="4.7625" width="0.3" layer="1"/>
+<wire x1="34.925" y1="14.9225" x2="32.7025" y2="12.7" width="0.3" layer="1"/>
+<wire x1="34.925" y1="14.9225" x2="35.0012" y2="14.9606" width="0.3" layer="1"/>
 </signal>
 <signal name="N$11" class="1">
 <contactref element="S3" pad="3"/>
 <contactref element="BT-IO" pad="2"/>
-<wire x1="27.94" y1="2.54" x2="26.1112" y2="14.9606" width="0" layer="19" extent="1-1"/>
+<wire x1="27.94" y1="3.4925" x2="27.94" y2="2.54" width="0.3" layer="1"/>
+<wire x1="23.8125" y1="7.62" x2="27.94" y2="3.4925" width="0.3" layer="1"/>
+<wire x1="23.8125" y1="12.7" x2="23.8125" y2="7.62" width="0.3" layer="1"/>
+<wire x1="26.035" y1="14.9225" x2="23.8125" y2="12.7" width="0.3" layer="1"/>
+<wire x1="26.035" y1="14.9225" x2="26.1112" y2="14.9606" width="0.3" layer="1"/>
 </signal>
 <signal name="N$12" class="1">
 <contactref element="S2" pad="3"/>
 <contactref element="BT-IO" pad="3"/>
-<wire x1="25.4" y1="2.54" x2="17.2212" y2="14.9606" width="0" layer="19" extent="1-1"/>
+<wire x1="25.4" y1="3.4925" x2="25.4" y2="2.54" width="0.3" layer="16"/>
+<wire x1="21.9075" y1="6.985" x2="25.4" y2="3.4925" width="0.3" layer="16"/>
+<wire x1="21.9075" y1="11.43" x2="21.9075" y2="6.985" width="0.3" layer="16"/>
+<wire x1="20.6375" y1="12.7" x2="21.9075" y2="11.43" width="0.3" layer="16"/>
+<wire x1="18.415" y1="12.7" x2="20.6375" y2="12.7" width="0.3" layer="16"/>
+<wire x1="17.145" y1="13.97" x2="18.415" y2="12.7" width="0.3" layer="16"/>
+<wire x1="17.145" y1="14.9225" x2="17.145" y2="13.97" width="0.3" layer="16"/>
+<wire x1="17.145" y1="14.9225" x2="17.2212" y2="14.9606" width="0.3" layer="16"/>
 </signal>
 <signal name="N$1">
 <contactref element="D1" pad="A"/>
 <contactref element="R3-220" pad="2"/>
-<wire x1="26.822" y1="63.5" x2="30.48" y2="63.5" width="0" layer="19" extent="1-1"/>
+<wire x1="28.575" y1="63.5" x2="26.822" y2="63.5" width="0.762" layer="1"/>
+<wire x1="28.8925" y1="63.8175" x2="28.575" y2="63.5" width="0.762" layer="1"/>
+<wire x1="30.1625" y1="63.8175" x2="28.8925" y2="63.8175" width="0.762" layer="1"/>
+<wire x1="30.48" y1="63.5" x2="30.1625" y2="63.8175" width="0.762" layer="1"/>
 </signal>
 <signal name="N$5">
 <contactref element="R3-220" pad="1"/>
 <contactref element="BT-IO" pad="4"/>
-<wire x1="22.86" y1="2.54" x2="23.978" y2="63.5" width="0" layer="19" extent="1-1"/>
+<wire x1="24.13" y1="16.51" x2="24.13" y2="63.5" width="0.762" layer="1"/>
+<wire x1="22.225" y1="14.605" x2="24.13" y2="16.51" width="0.762" layer="1"/>
+<wire x1="22.225" y1="5.3975" x2="22.225" y2="14.605" width="0.762" layer="1"/>
+<wire x1="21.59" y1="4.7625" x2="22.225" y2="5.3975" width="0.762" layer="1"/>
+<wire x1="21.59" y1="4.1275" x2="21.59" y2="4.7625" width="0.762" layer="1"/>
+<wire x1="22.86" y1="2.8575" x2="21.59" y2="4.1275" width="0.762" layer="1"/>
+<wire x1="22.86" y1="2.54" x2="22.86" y2="2.8575" width="0.762" layer="1"/>
+<wire x1="24.13" y1="63.5" x2="23.978" y2="63.5" width="0.762" layer="1"/>
 </signal>
 </signals>
