File: eagle/PCB/PCB 1d.brd (EAGLE design)
At the start: 45 x 75 mm, 29 parts

Commit message: PCB updates
Routing:
- net GND: track 2.99 -> 1.09 mm
Changed lines of the file:
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@@
 <drawing>
 <settings>
-<setting alwaysvectorfont="yes"/>
+<setting alwaysvectorfont="no"/>
 <setting verticaltext="up"/>
 </settings>
@@
 <wire x1="28.2575" y1="63.5" x2="27.23" y2="63.63" width="0.762" layer="1"/>
 <contactref element="MINIMOSD" pad="VGND1"/>
-<wire x1="17.78" y1="15.5476" x2="17.78" y2="15.24" width="0.1524" layer="1"/>
-<wire x1="16.8176" y1="16.51" x2="16.8176" y2="16.11135625" width="0.1524" layer="1"/>
-<wire x1="16.8176" y1="16.11135625" x2="17.38135625" y2="15.5476" width="0.1524" layer="1"/>
-<wire x1="17.38135625" y1="15.5476" x2="17.78" y2="15.5476" width="0.1524" layer="1"/>
 <via x="15.24" y="16.51" extent="1-16" drill="0.35"/>
 <via x="30.48" y="16.51" extent="1-16" drill="0.35"/>

Commit message: case work
Parts:
- moved DC-005 1.27 mm to (7.62, 7.62)
Routing:
- net +: track 6.10 -> 7.37 mm
Changed lines of the file:
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@@
 <board>
 <plain>
-<wire x1="0" y1="74.9808" x2="0" y2="0" width="0" layer="20" locked="yes"/>
+<wire x1="0" y1="74.9808" x2="0" y2="0" width="0" layer="20"/>
 <wire x1="0" y1="0" x2="44.9834" y2="0" width="0" layer="20" locked="yes"/>
 <wire x1="44.9834" y1="0" x2="44.9834" y2="74.9808" width="0" layer="20" locked="yes"/>
@@
 <attribute name="VALUE" x="19.05" y="2.54" size="0.0254" layer="27"/>
 </element>
-<element name="DC-005" library="con-jack" library_urn="urn:adsk.eagle:library:154" package="DCJ0202" package3d_urn="urn:adsk.eagle:package:7491/1" value="DCJ0202" x="7.62" y="8.89" smashed="yes">
-<attribute name="MF" value="" x="7.62" y="8.89" size="1.778" layer="27" display="off"/>
-<attribute name="MPN" value="" x="7.62" y="8.89" size="1.778" layer="27" display="off"/>
-<attribute name="NAME" x="5.08" y="2.54" size="1.27" layer="25"/>
-<attribute name="OC_FARNELL" value="unknown" x="7.62" y="8.89" size="1.778" layer="27" display="off"/>
-<attribute name="OC_NEWARK" value="unknown" x="7.62" y="8.89" size="1.778" layer="27" display="off"/>
-<attribute name="VALUE" x="13.97" y="0" size="1.27" layer="27" rot="R90"/>
+<element name="DC-005" library="con-jack" library_urn="urn:adsk.eagle:library:154" package="DCJ0202" package3d_urn="urn:adsk.eagle:package:7491/1" value="DCJ0202" x="7.62" y="7.62" smashed="yes">
+<attribute name="MF" value="" x="7.62" y="7.62" size="1.778" layer="27" display="off"/>
+<attribute name="MPN" value="" x="7.62" y="7.62" size="1.778" layer="27" display="off"/>
+<attribute name="NAME" x="5.08" y="1.27" size="1.27" layer="25"/>
+<attribute name="OC_FARNELL" value="unknown" x="7.62" y="7.62" size="1.778" layer="27" display="off"/>
+<attribute name="OC_NEWARK" value="unknown" x="7.62" y="7.62" size="1.778" layer="27" display="off"/>
+<attribute name="VALUE" x="13.97" y="-1.27" size="1.27" layer="27" rot="R90"/>
 </element>
 <element name="+IN" library="wirepad" library_urn="urn:adsk.eagle:library:412" package="2,54/1,1" package3d_urn="urn:adsk.eagle:package:30836/1" value="" x="3.81" y="16.51" smashed="yes" rot="R270">
@@
 <contactref element="+IN" pad="1"/>
 <contactref element="DC-005" pad="1"/>
-<wire x1="7.62" y1="12.7" x2="7.62" y2="11.99" width="0.762" layer="1"/>
+<wire x1="7.62" y1="12.7" x2="7.62" y2="10.72" width="0.762" layer="1"/>
 <wire x1="3.81" y1="16.51" x2="7.62" y2="12.7" width="0.762" layer="1"/>
 </signal>

Commit message: PCB and Case changes
Parts:
- removed A1: TPTP20SQ, testpad:TP20SQ
- added DVR_LED: TPTP20SQ, testpad:TP20SQ
- added U$2: (no value), holes:5,0
- moved DC-005 1.27 mm to (7.62, 8.89)
- renumbered DVR/MODULE-IO to MODULE-IO
Connections:
- net N$1: now also DVR_LED.TP; no longer A1.TP
Routing:
- net N$1: track 5.76 -> 18.8 mm
- net BEC-5V: track 74.7 -> 77.9 mm, vias 1 -> 2
- net +: track 7.37 -> 6.10 mm
- net SDA: track 46.8 -> 47.7 mm
- net SCL: track 54.7 -> 55.5 mm
Other:
- board text added: "DVR"
- board text added: "GND"
- board text added: "K1"
- board text added: "K2"
- board text added: "K3"
- board text added: "VID"
- board text added: "VIDin"
- board text removed: "D5"
- board text removed: "D6"
- board text removed: "D7"
- board text removed: "VIN/DVR"
- board text removed: "Vout"

Commit message: Case work and tiny PCB changes
Parts:
- moved DC-005 1.27 mm to (7.62, 7.62)
Routing:
- net +: track 6.10 -> 7.37 mm
Changed lines of the file:
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@@
 <attribute name="VALUE" x="19.05" y="2.54" size="0.0254" layer="27"/>
 </element>
-<element name="DC-005" library="con-jack" library_urn="urn:adsk.eagle:library:154" package="DCJ0202" package3d_urn="urn:adsk.eagle:package:7491/1" value="DCJ0202" x="7.62" y="8.89" smashed="yes">
-<attribute name="MF" value="" x="7.62" y="8.89" size="1.778" layer="27" display="off"/>
-<attribute name="MPN" value="" x="7.62" y="8.89" size="1.778" layer="27" display="off"/>
-<attribute name="NAME" x="5.08" y="2.54" size="1.27" layer="25"/>
-<attribute name="OC_FARNELL" value="unknown" x="7.62" y="8.89" size="1.778" layer="27" display="off"/>
-<attribute name="OC_NEWARK" value="unknown" x="7.62" y="8.89" size="1.778" layer="27" display="off"/>
-<attribute name="VALUE" x="13.97" y="0" size="1.27" layer="27" rot="R90"/>
+<element name="DC-005" library="con-jack" library_urn="urn:adsk.eagle:library:154" package="DCJ0202" package3d_urn="urn:adsk.eagle:package:7491/1" value="DCJ0202" x="7.62" y="7.62" smashed="yes">
+<attribute name="MF" value="" x="7.62" y="7.62" size="1.778" layer="27" display="off"/>
+<attribute name="MPN" value="" x="7.62" y="7.62" size="1.778" layer="27" display="off"/>
+<attribute name="NAME" x="5.08" y="1.27" size="1.27" layer="25"/>
+<attribute name="OC_FARNELL" value="unknown" x="7.62" y="7.62" size="1.778" layer="27" display="off"/>
+<attribute name="OC_NEWARK" value="unknown" x="7.62" y="7.62" size="1.778" layer="27" display="off"/>
+<attribute name="VALUE" x="13.97" y="-1.27" size="1.27" layer="27" rot="R90"/>
 </element>
 <element name="+IN" library="wirepad" library_urn="urn:adsk.eagle:library:412" package="2,54/1,1" package3d_urn="urn:adsk.eagle:package:30836/1" value="" x="3.81" y="16.51" smashed="yes" rot="R270">
@@
 <contactref element="+IN" pad="1"/>
 <contactref element="DC-005" pad="1"/>
-<wire x1="7.62" y1="12.7" x2="7.62" y2="11.99" width="0.762" layer="1"/>
+<wire x1="7.62" y1="12.7" x2="7.62" y2="10.72" width="0.762" layer="1"/>
 <wire x1="3.81" y1="16.51" x2="7.62" y2="12.7" width="0.762" layer="1"/>
 </signal>
