File: eagle/PCB/PCB 2d.brd (EAGLE design)
At the start: 45 x 75 mm, 17 parts

Commit message: PCB and Case changes
Parts:
- moved VSW_O 12.8 mm to (24.1, 57.1), flipped to the bottom
- moved R3-220 11.7 mm to (31.8, 58.4), turned to 180 degrees
- moved VSW 5.08 mm to (20.3, 69.8), flipped to the bottom
- turned D1 to 180 degrees
Routing:
- net VIDOUT: track 29.6 -> 18.8 mm
- net N$5: track 70.9 -> 61.6 mm
- net N$8: track 32.7 -> 24.7 mm
- net N$4: track 50.9 -> 53.6 mm
- net N$3: track 18.9 -> 21.2 mm
- net N$10: track 31.1 -> 29.1 mm
- net N$1: track 7.55 -> 6.47 mm

Commit message: Small PCB change
Parts:
- moved VSW_O 12.7 mm to (11.4, 57.1), flipped to the top
- moved VSW 5.08 mm to (15.2, 69.8), flipped to the top
Routing:
- net VIDOUT: track 18.8 -> 30.5 mm
- net N$8: track 24.7 -> 32.7 mm
- net N$4: track 53.6 -> 50.9 mm
- net N$10: track 29.1 -> 31.4 mm
Changed lines of the file:
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@@
 <layer number="20" name="Dimension" color="24" fill="1" visible="yes" active="yes"/>
 <layer number="21" name="tPlace" color="7" fill="1" visible="yes" active="yes"/>
-<layer number="22" name="bPlace" color="7" fill="1" visible="yes" active="yes"/>
+<layer number="22" name="bPlace" color="7" fill="1" visible="no" active="yes"/>
 <layer number="23" name="tOrigins" color="15" fill="1" visible="yes" active="yes"/>
-<layer number="24" name="bOrigins" color="15" fill="1" visible="yes" active="yes"/>
+<layer number="24" name="bOrigins" color="15" fill="1" visible="no" active="yes"/>
 <layer number="25" name="tNames" color="7" fill="1" visible="yes" active="yes"/>
-<layer number="26" name="bNames" color="7" fill="1" visible="yes" active="yes"/>
+<layer number="26" name="bNames" color="7" fill="1" visible="no" active="yes"/>
 <layer number="27" name="tValues" color="7" fill="1" visible="no" active="yes"/>
 <layer number="28" name="bValues" color="7" fill="1" visible="no" active="yes"/>
@@
 <layer number="38" name="bTest" color="7" fill="1" visible="no" active="yes"/>
 <layer number="39" name="tKeepout" color="4" fill="11" visible="yes" active="yes"/>
-<layer number="40" name="bKeepout" color="1" fill="11" visible="yes" active="yes"/>
+<layer number="40" name="bKeepout" color="1" fill="11" visible="no" active="yes"/>
 <layer number="41" name="tRestrict" color="4" fill="10" visible="yes" active="yes"/>
-<layer number="42" name="bRestrict" color="1" fill="10" visible="yes" active="yes"/>
+<layer number="42" name="bRestrict" color="1" fill="10" visible="no" active="yes"/>
 <layer number="43" name="vRestrict" color="2" fill="10" visible="no" active="yes"/>
 <layer number="44" name="Drills" color="7" fill="1" visible="no" active="yes"/>
@@
 <layer number="50" name="dxf" color="7" fill="1" visible="no" active="no"/>
 <layer number="51" name="tDocu" color="7" fill="1" visible="yes" active="yes"/>
-<layer number="52" name="bDocu" color="7" fill="1" visible="yes" active="yes"/>
+<layer number="52" name="bDocu" color="7" fill="1" visible="no" active="yes"/>
 <layer number="53" name="tGND_GNDA" color="7" fill="9" visible="no" active="no"/>
 <layer number="54" name="bGND_GNDA" color="1" fill="9" visible="no" active="no"/>
@@
 </element>
 <element name="D9PWM" library="SparkFun-Connectors" library_urn="urn:adsk.eagle:library:513" package="1X01" package3d_urn="urn:adsk.eagle:package:38028/1" value="" x="41.91" y="62.23"/>
-<element name="VSW" library="SparkFun-Connectors" library_urn="urn:adsk.eagle:library:513" package="1X03" package3d_urn="urn:adsk.eagle:package:38063/1" value="" x="20.32" y="69.85" rot="MR0"/>
-<element name="VSW_O" library="SparkFun-Connectors" library_urn="urn:adsk.eagle:library:513" package="1X06" package3d_urn="urn:adsk.eagle:package:38009/1" value="" x="24.13" y="57.15" rot="MR0">
-<attribute name="PROD_ID" value="CONN-08437" x="24.13" y="57.15" size="1.778" layer="28" rot="MR0" display="off"/>
+<element name="VSW" library="SparkFun-Connectors" library_urn="urn:adsk.eagle:library:513" package="1X03" package3d_urn="urn:adsk.eagle:package:38063/1" value="" x="15.24" y="69.85"/>
+<element name="VSW_O" library="SparkFun-Connectors" library_urn="urn:adsk.eagle:library:513" package="1X06" package3d_urn="urn:adsk.eagle:package:38009/1" value="" x="11.43" y="57.15">
+<attribute name="PROD_ID" value="CONN-08437" x="11.43" y="57.15" size="1.778" layer="27" display="off"/>
 </element>
 </elements>
@@
 <contactref element="S1" pad="1"/>
 <wire x1="5.3975" y1="55.88" x2="3.81" y2="55.88" width="0.4" layer="16"/>
-<wire x1="12.3825" y1="62.865" x2="10.4775" y2="60.96" width="0.4" layer="16"/>
-<wire x1="10.4775" y1="60.96" x2="5.3975" y2="55.88" width="0.4" layer="16"/>
+<wire x1="12.3825" y1="62.865" x2="6.985" y2="57.4675" width="0.4" layer="16"/>
+<wire x1="6.985" y1="57.4675" x2="5.3975" y2="55.88" width="0.4" layer="16"/>
 <wire x1="12.7" y1="62.865" x2="12.3825" y2="62.865" width="0.4" layer="16"/>
 <wire x1="13.335" y1="63.5" x2="12.7" y2="62.865" width="0.4" layer="16"/>
 <wire x1="13.97" y1="63.5" x2="13.335" y2="63.5" width="0.4" layer="16"/>
 <contactref element="VSW_O" pad="5"/>
-<wire x1="13.97" y1="57.785" x2="13.97" y2="57.15" width="0.4" layer="16"/>
-<wire x1="10.795" y1="60.96" x2="13.97" y2="57.785" width="0.4" layer="16"/>
-<wire x1="10.4775" y1="60.96" x2="10.795" y2="60.96" width="0.4" layer="16"/>
+<wire x1="21.59" y1="56.515" x2="21.59" y2="57.15" width="0.4" layer="16"/>
+<wire x1="19.685" y1="54.61" x2="21.59" y2="56.515" width="0.4" layer="16"/>
+<wire x1="10.16" y1="54.61" x2="19.685" y2="54.61" width="0.4" layer="16"/>
+<wire x1="7.3025" y1="57.4675" x2="10.16" y2="54.61" width="0.4" layer="16"/>
+<wire x1="6.985" y1="57.4675" x2="7.3025" y2="57.4675" width="0.4" layer="16"/>
 </signal>
 <signal name="N$3" class="2">
@@
 <wire x1="5.3975" y1="58.42" x2="3.81" y2="58.42" width="0.4" layer="1"/>
 <wire x1="7.3025" y1="60.325" x2="5.3975" y2="58.42" width="0.4" layer="1"/>
-<wire x1="14.9225" y1="60.325" x2="7.3025" y2="60.325" width="0.4" layer="1"/>
-<wire x1="16.51" y1="61.9125" x2="15.5575" y2="60.96" width="0.4" layer="1"/>
-<wire x1="15.5575" y1="60.96" x2="14.9225" y2="60.325" width="0.4" layer="1"/>
+<wire x1="14.9225" y1="60.325" x2="14.605" y2="60.325" width="0.4" layer="1"/>
+<wire x1="14.605" y1="60.325" x2="7.3025" y2="60.325" width="0.4" layer="1"/>
+<wire x1="16.51" y1="61.9125" x2="14.9225" y2="60.325" width="0.4" layer="1"/>
 <wire x1="16.51" y1="63.5" x2="16.51" y2="61.9125" width="0.4" layer="1"/>
 <contactref element="VSW_O" pad="3"/>
-<wire x1="19.05" y1="57.785" x2="19.05" y2="57.15" width="0.4" layer="1"/>
-<wire x1="15.875" y1="60.96" x2="19.05" y2="57.785" width="0.4" layer="1"/>
-<wire x1="15.5575" y1="60.96" x2="15.875" y2="60.96" width="0.4" layer="1"/>
+<wire x1="16.51" y1="59.055" x2="16.51" y2="57.15" width="0.4" layer="1"/>
+<wire x1="16.1925" y1="59.3725" x2="16.51" y2="59.055" width="0.4" layer="1"/>
+<wire x1="16.1925" y1="60.0075" x2="16.1925" y2="59.3725" width="0.4" layer="1"/>
+<wire x1="15.24" y1="60.96" x2="16.1925" y2="60.0075" width="0.4" layer="1"/>
+<wire x1="14.605" y1="60.325" x2="15.24" y2="60.96" width="0.4" layer="1"/>
 </signal>
 <signal name="GND">
@@
 <contactref element="VSW" pad="2"/>
 <wire x1="17.78" y1="69.215" x2="17.78" y2="69.85" width="0.762" layer="16"/>
-<wire x1="16.51" y1="67.945" x2="17.78" y2="69.215" width="0.762" layer="16"/>
-<wire x1="16.51" y1="67.6275" x2="16.51" y2="67.945" width="0.762" layer="16"/>
-<wire x1="17.145" y1="66.9925" x2="16.51" y2="67.6275" width="0.762" layer="16"/>
-<wire x1="23.8125" y1="66.9925" x2="17.145" y2="66.9925" width="0.762" layer="16"/>
-<wire x1="33.9725" y1="56.8325" x2="23.8125" y2="66.9925" width="0.762" layer="16"/>
-<wire x1="39.37" y1="56.8325" x2="33.9725" y2="56.8325" width="0.762" layer="16"/>
+<wire x1="30.1625" y1="56.8325" x2="17.78" y2="69.215" width="0.762" layer="16"/>
+<wire x1="39.37" y1="56.8325" x2="30.1625" y2="56.8325" width="0.762" layer="16"/>
 </signal>
 <signal name="N$6" class="1">
@@
 <wire x1="19.05" y1="63.5" x2="19.05" y2="65.0875" width="0.4" layer="1"/>
 <contactref element="VSW_O" pad="1"/>
-<wire x1="24.13" y1="57.785" x2="24.13" y2="57.15" width="0.4" layer="1"/>
-<wire x1="21.2725" y1="60.6425" x2="24.13" y2="57.785" width="0.4" layer="1"/>
-<wire x1="21.2725" y1="62.5475" x2="21.2725" y2="60.6425" width="0.4" layer="1"/>
-<wire x1="20.6375" y1="63.1825" x2="21.2725" y2="62.5475" width="0.4" layer="1"/>
-<wire x1="19.3675" y1="63.1825" x2="20.6375" y2="63.1825" width="0.4" layer="1"/>
-<wire x1="19.05" y1="63.5" x2="19.3675" y2="63.1825" width="0.4" layer="1"/>
+<wire x1="11.43" y1="57.785" x2="11.43" y2="57.15" width="0.4" layer="16"/>
+<wire x1="13.97" y1="60.325" x2="11.43" y2="57.785" width="0.4" layer="16"/>
+<wire x1="17.4625" y1="60.325" x2="13.97" y2="60.325" width="0.4" layer="16"/>
+<wire x1="19.05" y1="61.9125" x2="17.4625" y2="60.325" width="0.4" layer="16"/>
+<wire x1="19.05" y1="63.5" x2="19.05" y2="61.9125" width="0.4" layer="16"/>
 </signal>
 <signal name="N$2" class="1">
@@
 <contactref element="VSW" pad="1"/>
 <contactref element="D9PWM" pad="1"/>
-<wire x1="20.6375" y1="69.85" x2="20.32" y2="69.85" width="0.762" layer="1"/>
-<wire x1="24.4475" y1="66.04" x2="20.6375" y2="69.85" width="0.762" layer="1"/>
-<wire x1="37.7825" y1="66.04" x2="24.4475" y2="66.04" width="0.762" layer="1"/>
-<wire x1="41.5925" y1="62.23" x2="37.7825" y2="66.04" width="0.762" layer="1"/>
+<wire x1="15.24" y1="70.8025" x2="15.24" y2="69.85" width="0.762" layer="1"/>
+<wire x1="15.5575" y1="71.12" x2="15.24" y2="70.8025" width="0.762" layer="1"/>
+<wire x1="15.5575" y1="71.4375" x2="15.5575" y2="71.12" width="0.762" layer="1"/>
+<wire x1="16.51" y1="72.39" x2="15.5575" y2="71.4375" width="0.762" layer="1"/>
+<wire x1="31.4325" y1="72.39" x2="16.51" y2="72.39" width="0.762" layer="1"/>
+<wire x1="41.5925" y1="62.23" x2="31.4325" y2="72.39" width="0.762" layer="1"/>
 <wire x1="41.91" y1="62.23" x2="41.5925" y2="62.23" width="0.762" layer="1"/>
 </signal>

Commit message: Case work and tiny PCB changes
Parts:
- moved VSW 1.27 mm to (16.5, 69.8)
- moved VSW_O 1.27 mm to (12.7, 57.1)
Routing:
- net N$4: track 50.9 -> 49.6 mm
- net N$10: track 31.4 -> 30.1 mm
- net VIDOUT: track 30.5 -> 31.3 mm
- net N$3: track 21.0 -> 21.5 mm
Changed lines of the file:
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@@
 </element>
 <element name="D9PWM" library="SparkFun-Connectors" library_urn="urn:adsk.eagle:library:513" package="1X01" package3d_urn="urn:adsk.eagle:package:38028/1" value="" x="41.91" y="62.23"/>
-<element name="VSW" library="SparkFun-Connectors" library_urn="urn:adsk.eagle:library:513" package="1X03" package3d_urn="urn:adsk.eagle:package:38063/1" value="" x="15.24" y="69.85"/>
-<element name="VSW_O" library="SparkFun-Connectors" library_urn="urn:adsk.eagle:library:513" package="1X06" package3d_urn="urn:adsk.eagle:package:38009/1" value="" x="11.43" y="57.15">
-<attribute name="PROD_ID" value="CONN-08437" x="11.43" y="57.15" size="1.778" layer="27" display="off"/>
+<element name="VSW" library="SparkFun-Connectors" library_urn="urn:adsk.eagle:library:513" package="1X03" package3d_urn="urn:adsk.eagle:package:38063/1" value="" x="16.51" y="69.85"/>
+<element name="VSW_O" library="SparkFun-Connectors" library_urn="urn:adsk.eagle:library:513" package="1X06" package3d_urn="urn:adsk.eagle:package:38009/1" value="" x="12.7" y="57.15">
+<attribute name="PROD_ID" value="CONN-08437" x="12.7" y="57.15" size="1.778" layer="27" display="off"/>
 </element>
 </elements>
@@
 <wire x1="13.97" y1="63.5" x2="13.335" y2="63.5" width="0.4" layer="16"/>
 <contactref element="VSW_O" pad="5"/>
-<wire x1="21.59" y1="56.515" x2="21.59" y2="57.15" width="0.4" layer="16"/>
+<wire x1="21.59" y1="56.515" x2="22.86" y2="57.15" width="0.4" layer="16"/>
 <wire x1="19.685" y1="54.61" x2="21.59" y2="56.515" width="0.4" layer="16"/>
 <wire x1="10.16" y1="54.61" x2="19.685" y2="54.61" width="0.4" layer="16"/>
@@
 <wire x1="16.51" y1="63.5" x2="16.51" y2="61.9125" width="0.4" layer="1"/>
 <contactref element="VSW_O" pad="3"/>
-<wire x1="16.51" y1="59.055" x2="16.51" y2="57.15" width="0.4" layer="1"/>
-<wire x1="16.1925" y1="59.3725" x2="16.51" y2="59.055" width="0.4" layer="1"/>
-<wire x1="16.1925" y1="60.0075" x2="16.1925" y2="59.3725" width="0.4" layer="1"/>
-<wire x1="15.24" y1="60.96" x2="16.1925" y2="60.0075" width="0.4" layer="1"/>
+<wire x1="17.78" y1="57.785" x2="17.78" y2="57.15" width="0.4" layer="1"/>
+<wire x1="16.51" y1="59.055" x2="17.78" y2="57.785" width="0.4" layer="1"/>
+<wire x1="16.51" y1="59.69" x2="16.51" y2="59.055" width="0.4" layer="1"/>
+<wire x1="15.24" y1="60.96" x2="16.51" y2="59.69" width="0.4" layer="1"/>
 <wire x1="14.605" y1="60.325" x2="15.24" y2="60.96" width="0.4" layer="1"/>
 </signal>
@@
 <wire x1="41.91" y1="59.69" x2="41.275" y2="59.69" width="0.762" layer="16"/>
 <contactref element="VSW" pad="2"/>
-<wire x1="17.78" y1="69.215" x2="17.78" y2="69.85" width="0.762" layer="16"/>
-<wire x1="30.1625" y1="56.8325" x2="17.78" y2="69.215" width="0.762" layer="16"/>
-<wire x1="39.37" y1="56.8325" x2="30.1625" y2="56.8325" width="0.762" layer="16"/>
+<wire x1="19.05" y1="69.215" x2="19.05" y2="69.85" width="0.762" layer="16"/>
+<wire x1="31.4325" y1="56.8325" x2="19.05" y2="69.215" width="0.762" layer="16"/>
+<wire x1="39.37" y1="56.8325" x2="31.4325" y2="56.8325" width="0.762" layer="16"/>
 </signal>
 <signal name="N$6" class="1">
@@
 <wire x1="19.05" y1="63.5" x2="19.05" y2="65.0875" width="0.4" layer="1"/>
 <contactref element="VSW_O" pad="1"/>
-<wire x1="11.43" y1="57.785" x2="11.43" y2="57.15" width="0.4" layer="16"/>
-<wire x1="13.97" y1="60.325" x2="11.43" y2="57.785" width="0.4" layer="16"/>
-<wire x1="17.4625" y1="60.325" x2="13.97" y2="60.325" width="0.4" layer="16"/>
+<wire x1="12.7" y1="57.785" x2="12.7" y2="57.15" width="0.4" layer="16"/>
+<wire x1="15.24" y1="60.325" x2="12.7" y2="57.785" width="0.4" layer="16"/>
+<wire x1="17.4625" y1="60.325" x2="15.24" y2="60.325" width="0.4" layer="16"/>
 <wire x1="19.05" y1="61.9125" x2="17.4625" y2="60.325" width="0.4" layer="16"/>
 <wire x1="19.05" y1="63.5" x2="19.05" y2="61.9125" width="0.4" layer="16"/>
@@
 <contactref element="VSW" pad="1"/>
 <contactref element="D9PWM" pad="1"/>
-<wire x1="15.24" y1="70.8025" x2="15.24" y2="69.85" width="0.762" layer="1"/>
-<wire x1="15.5575" y1="71.12" x2="15.24" y2="70.8025" width="0.762" layer="1"/>
-<wire x1="15.5575" y1="71.4375" x2="15.5575" y2="71.12" width="0.762" layer="1"/>
-<wire x1="16.51" y1="72.39" x2="15.5575" y2="71.4375" width="0.762" layer="1"/>
-<wire x1="31.4325" y1="72.39" x2="16.51" y2="72.39" width="0.762" layer="1"/>
-<wire x1="41.5925" y1="62.23" x2="31.4325" y2="72.39" width="0.762" layer="1"/>
+<wire x1="41.5925" y1="62.23" x2="32.0675" y2="71.755" width="0.762" layer="1"/>
+<wire x1="32.0675" y1="71.755" x2="31.4325" y2="72.39" width="0.762" layer="1"/>
 <wire x1="41.91" y1="62.23" x2="41.5925" y2="62.23" width="0.762" layer="1"/>
+<wire x1="16.51" y1="70.8025" x2="16.51" y2="69.85" width="0.762" layer="1"/>
+<wire x1="16.8275" y1="71.12" x2="16.51" y2="70.8025" width="0.762" layer="1"/>
+<wire x1="16.8275" y1="71.4375" x2="16.8275" y2="71.12" width="0.762" layer="1"/>
+<wire x1="17.78" y1="72.39" x2="16.8275" y2="71.4375" width="0.762" layer="1"/>
+<wire x1="28.575" y1="72.39" x2="17.78" y2="72.39" width="0.762" layer="1"/>
+<wire x1="30.1625" y1="70.8025" x2="28.575" y2="72.39" width="0.762" layer="1"/>
+<wire x1="31.115" y1="70.8025" x2="30.1625" y2="70.8025" width="0.762" layer="1"/>
+<wire x1="32.0675" y1="71.755" x2="31.115" y2="70.8025" width="0.762" layer="1"/>
 </signal>
 </signals>
