File: PCB Files/EAGLE PCB/PCB 1d.brd (EAGLE design)
At the start: 45 x 75 mm, 30 parts

Commit message: Updated PCBs
• Round edges
• Covered vias on PCB1
• OLED pin swap (VCC <> GND) on PCB2
Other:
- outline, holes or cut-outs redrawn
Changed lines of the file:
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@@
 <board>
 <plain>
-<wire x1="0" y1="74.9808" x2="0" y2="0" width="0" layer="20"/>
-<wire x1="0" y1="0" x2="44.9834" y2="0" width="0" layer="20" locked="yes"/>
-<wire x1="44.9834" y1="0" x2="44.9834" y2="74.9808" width="0" layer="20" locked="yes"/>
-<wire x1="44.9834" y1="74.9808" x2="0" y2="74.9808" width="0" layer="20" locked="yes"/>
+<wire x1="41.9421875" y1="74.9808" x2="4.422415625" y2="74.9808" width="0" layer="20"/>
+<wire x1="4.422415625" y1="74.9808" x2="0" y2="70.558384375" width="0" layer="20" curve="90"/>
+<wire x1="0" y1="70.558384375" x2="0" y2="4.33604375" width="0" layer="20"/>
+<wire x1="0" y1="4.33604375" x2="4.33604375" y2="0" width="0" layer="20" curve="90"/>
+<wire x1="4.33604375" y1="0" x2="42.01600625" y2="0" width="0" layer="20"/>
+<wire x1="42.01600625" y1="0" x2="44.9834" y2="2.96739375" width="0" layer="20" curve="90"/>
+<wire x1="44.9834" y1="2.96739375" x2="44.9834" y2="71.9395875" width="0" layer="20"/>
+<wire x1="44.9834" y1="71.9395875" x2="41.9421875" y2="74.9808" width="0" layer="20" curve="90"/>
 <text x="39.37" y="50.8" size="0.889" layer="25" rot="R90">SDA</text>
 <text x="39.37" y="53.34" size="0.889" layer="25" rot="R90">SCL</text>
@@
 <param name="mlMinCreamFrame" value="0mil"/>
 <param name="mlMaxCreamFrame" value="0mil"/>
-<param name="mlViaStopLimit" value="0mil"/>
+<param name="mlViaStopLimit" value="2mm"/>
 <param name="srRoundness" value="0"/>
 <param name="srMinRoundness" value="0mil"/>
@@
 packages will not be understood (or retained) with this version.
 </note>
-<note version="8.5" severity="warning">
-Since Version 8.5, EAGLE supports locking for holes, vias, wires and polygons.
-The locking property on all objects of these types will not be understood in this version.
-</note>
 </compatibility>

Commit message: New PCB revision (added a cap)
Parts:
- added C1: (no value), rcl:C1206K
Connections:
- net GND: now also C1.2, U$1.GND1
- net VSENS: now also C1.1
Routing:
- net VSENS: track 16.7 -> 18.8 mm
- net GND: vias 2 -> 8
Other:
- board text added: "POCKET-GROUNDSTATION | PCB1 | REV2"
- board text removed: "POCKET-GROUNDSTATION | PCB1 | REV1"
Changed lines of the file:
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@@
 <grid distance="50" unitdist="mil" unit="mil" style="dots" multiple="1" display="yes" altdistance="5" altunitdist="mil" altunit="mil"/>
 <layers>
-<layer number="1" name="Top" color="4" fill="1" visible="yes" active="yes"/>
+<layer number="1" name="Top" color="4" fill="1" visible="no" active="yes"/>
 <layer number="2" name="Route2" color="1" fill="3" visible="no" active="no"/>
 <layer number="3" name="Route3" color="4" fill="3" visible="no" active="no"/>
@@
 <layer number="19" name="Unrouted" color="6" fill="1" visible="yes" active="yes"/>
 <layer number="20" name="Dimension" color="24" fill="1" visible="yes" active="yes"/>
-<layer number="21" name="tPlace" color="7" fill="1" visible="yes" active="yes"/>
-<layer number="22" name="bPlace" color="7" fill="1" visible="no" active="yes"/>
-<layer number="23" name="tOrigins" color="15" fill="1" visible="yes" active="yes"/>
-<layer number="24" name="bOrigins" color="15" fill="1" visible="no" active="yes"/>
-<layer number="25" name="tNames" color="7" fill="1" visible="yes" active="yes"/>
-<layer number="26" name="bNames" color="7" fill="1" visible="no" active="yes"/>
+<layer number="21" name="tPlace" color="7" fill="1" visible="no" active="yes"/>
+<layer number="22" name="bPlace" color="7" fill="1" visible="yes" active="yes"/>
+<layer number="23" name="tOrigins" color="15" fill="1" visible="no" active="yes"/>
+<layer number="24" name="bOrigins" color="15" fill="1" visible="yes" active="yes"/>
+<layer number="25" name="tNames" color="7" fill="1" visible="no" active="yes"/>
+<layer number="26" name="bNames" color="7" fill="1" visible="yes" active="yes"/>
 <layer number="27" name="tValues" color="7" fill="1" visible="no" active="yes"/>
 <layer number="28" name="bValues" color="7" fill="1" visible="no" active="yes"/>
@@
 <layer number="37" name="tTest" color="7" fill="1" visible="no" active="yes"/>
 <layer number="38" name="bTest" color="7" fill="1" visible="no" active="yes"/>
-<layer number="39" name="tKeepout" color="4" fill="11" visible="yes" active="yes"/>
-<layer number="40" name="bKeepout" color="1" fill="11" visible="no" active="yes"/>
-<layer number="41" name="tRestrict" color="4" fill="10" visible="yes" active="yes"/>
-<layer number="42" name="bRestrict" color="1" fill="10" visible="no" active="yes"/>
+<layer number="39" name="tKeepout" color="4" fill="11" visible="no" active="yes"/>
+<layer number="40" name="bKeepout" color="1" fill="11" visible="yes" active="yes"/>
+<layer number="41" name="tRestrict" color="4" fill="10" visible="no" active="yes"/>
+<layer number="42" name="bRestrict" color="1" fill="10" visible="yes" active="yes"/>
 <layer number="43" name="vRestrict" color="2" fill="10" visible="no" active="yes"/>
 <layer number="44" name="Drills" color="7" fill="1" visible="no" active="yes"/>
@@
 <layer number="49" name="Reference" color="7" fill="1" visible="no" active="yes"/>
 <layer number="50" name="dxf" color="7" fill="1" visible="no" active="no"/>
-<layer number="51" name="tDocu" color="7" fill="1" visible="yes" active="yes"/>
-<layer number="52" name="bDocu" color="7" fill="1" visible="no" active="yes"/>
+<layer number="51" name="tDocu" color="7" fill="1" visible="no" active="yes"/>
+<layer number="52" name="bDocu" color="7" fill="1" visible="yes" active="yes"/>
 <layer number="53" name="tGND_GNDA" color="7" fill="9" visible="no" active="no"/>
 <layer number="54" name="bGND_GNDA" color="1" fill="9" visible="no" active="no"/>
@@
 <text x="2.54" y="19.05" size="1.016" layer="26" rot="MR90">&lt; To switch</text>
 <text x="12.7" y="1.27" size="1.016" layer="26" rot="MR0">&lt; From switch</text>
-<text x="43.18" y="48.26" size="1.27" layer="26" rot="MR270">POCKET-GROUNDSTATION | PCB1 | REV1</text>
+<text x="43.18" y="48.26" size="1.27" layer="26" rot="MR270">POCKET-GROUNDSTATION | PCB1 | REV2</text>
 <text x="1.27" y="52.07" size="0.889" layer="26" rot="MR90">VID</text>
 <text x="1.27" y="46.99" size="0.889" layer="26" rot="MR90">G</text>
@@
 <element name="PWM" library="SparkFun-Connectors" library_urn="urn:adsk.eagle:library:513" package="1X01" package3d_urn="urn:adsk.eagle:package:38028/1" value="" x="41.91" y="62.23"/>
 <element name="U$2" library="holes" library_urn="urn:adsk.eagle:library:237" package="5,0" package3d_urn="urn:adsk.eagle:package:14276/1" value="" x="22.86" y="49.53"/>
+<element name="C1" library="rcl" library_urn="urn:adsk.eagle:library:334" package="C1206K" package3d_urn="urn:adsk.eagle:package:23682/2" value="" x="31.75" y="30.48">
+<attribute name="SPICEPREFIX" value="C" x="31.75" y="30.48" size="1.778" layer="27" display="off"/>
+</element>
 </elements>
 <signals>
@@
 <via x="15.24" y="16.51" extent="1-16" drill="0.35"/>
 <via x="30.48" y="16.51" extent="1-16" drill="0.35"/>
+<contactref element="C1" pad="2"/>
+<contactref element="U$1" pad="GND1"/>
+<via x="27.94" y="40.64" extent="1-16" drill="0.35"/>
+<via x="39.37" y="3.81" extent="1-16" drill="0.35"/>
+<via x="2.54" y="7.62" extent="1-16" drill="0.35"/>
+<via x="35.56" y="60.96" extent="1-16" drill="0.35"/>
+<via x="5.08" y="68.58" extent="1-16" drill="0.35"/>
+<via x="26.67" y="43.18" extent="1-16" drill="0.35"/>
 </signal>
 <signal name="+5VFTDI" class="1">
@@
 <wire x1="25.27" y1="27.94" x2="17.91" y2="27.94" width="0.762" layer="1"/>
 <wire x1="29.21" y1="32.385" x2="29.21" y2="35.56" width="0.762" layer="1"/>
-<wire x1="25.0825" y1="28.2575" x2="29.21" y2="32.385" width="0.762" layer="1"/>
+<wire x1="25.0825" y1="28.2575" x2="28.73375" y2="31.90875" width="0.762" layer="1"/>
+<wire x1="28.73375" y1="31.90875" x2="29.21" y2="32.385" width="0.762" layer="1"/>
 <wire x1="25.0825" y1="28.2575" x2="25.27" y2="27.94" width="0.762" layer="1"/>
+<contactref element="C1" pad="1"/>
+<wire x1="28.73375" y1="31.90875" x2="30.1625" y2="30.48" width="0.762" layer="1"/>
+<wire x1="30.1625" y1="30.48" x2="30.25" y2="30.48" width="0.762" layer="1"/>
 </signal>
 <signal name="D5" class="1">
@@
 <contactref element="U$1" pad="D13"/>
 <contactref element="BT-BRIDGE" pad="4"/>
-<wire x1="31.75" y1="32.385" x2="31.75" y2="35.56" width="0.4" layer="1"/>
-<wire x1="43.4975" y1="20.6375" x2="31.75" y2="32.385" width="0.4" layer="1"/>
-<wire x1="43.4975" y1="16.8275" x2="43.4975" y2="20.6375" width="0.4" layer="1"/>
 <wire x1="36.5125" y1="9.8425" x2="43.4975" y2="16.8275" width="0.4" layer="1"/>
 <wire x1="30.1625" y1="9.8425" x2="36.5125" y2="9.8425" width="0.4" layer="1"/>
 <wire x1="22.86" y1="2.54" x2="30.1625" y2="9.8425" width="0.4" layer="1"/>
+<wire x1="31.75" y1="34.6075" x2="31.75" y2="35.56" width="0.4" layer="1"/>
+<wire x1="37.1475" y1="29.21" x2="31.75" y2="34.6075" width="0.4" layer="1"/>
+<wire x1="37.1475" y1="26.9875" x2="37.1475" y2="29.21" width="0.4" layer="1"/>
+<wire x1="43.4975" y1="20.6375" x2="37.1475" y2="26.9875" width="0.4" layer="1"/>
+<wire x1="43.4975" y1="16.8275" x2="43.4975" y2="20.6375" width="0.4" layer="1"/>
 </signal>
 <signal name="8V">
