File: PCB Files/EAGLE PCB/PCB 1d.sch (EAGLE design)
At the start: 29 parts

Commit message: New PCB revision (added a cap)
Parts:
- added C1: (no value), rcl:C-EUC1206K
Connections:
- net GND: now also C1.2, U$1.GND2
- net VSENS: now also C1.1
